File: multiplier.kicad_sch (KiCad schematic)
At the start: 4 parts, among them U36 4081, U37 4081, U38 4081, U39 4069

Commit message: Add files via upload
Waiting for approval
Other:
- sheet FullAdder ports: added xor_out; removed none
- sheet FullAdder1 ports: added xor_out; removed none
- sheet FullAdder2 ports: added xor_out; removed none
- sheet FullAdder3 ports: added xor_out; removed none
- sheet FullAdder4 ports: added xor_out; removed none
- sheet FullAdder5 ports: added xor_out; removed none
Changed lines of the file:
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@@
+			)
+		)
+		(pin "xor_out" output
+			(at 229.87 88.9 0)
+			(effects
+				(font
+					(size 1.27 1.27)
+				)
+				(justify right)
 			)
 		)
@@
 			)
 		)
+		(pin "xor_out" output
+			(at 151.13 66.04 0)
+			(effects
+				(font
+					(size 1.27 1.27)
+				)
+				(justify right)
+			)
+		)
 		(instances
 			(project "DTS"
@@
 			)
 		)
+		(pin "xor_out" output
+			(at 151.13 36.83 0)
+			(effects
+				(font
+					(size 1.27 1.27)
+				)
+				(justify right)
+			)
+		)
 		(instances
 			(project "DTS"
@@
 			)
 		)
+		(pin "xor_out" output
+			(at 228.6 60.96 0)
+			(effects
+				(font
+					(size 1.27 1.27)
+				)
+				(justify right)
+			)
+		)
 		(instances
 			(project "DTS"
@@
 			)
 		)
+		(pin "xor_out" output
+			(at 151.13 91.44 0)
+			(effects
+				(font
+					(size 1.27 1.27)
+				)
+				(justify right)
+			)
+		)
 		(instances
 			(project "DTS"
@@
 			)
 		)
+		(pin "xor_out" output
+			(at 228.6 36.83 0)
+			(effects
+				(font
+					(size 1.27 1.27)
+				)
+				(justify right)
+			)
+		)
