File: multiplier.kicad_sch (KiCad schematic)
At the start: 4 parts, among them U12 4081, U2 4081, U37 4069, U7 4081

Commit message: Add files via upload
Connections:
- net A0: now also U2.2
- net B0: now also U2.1
