File: multiplier.kicad_sch (KiCad schematic)
At the start: 4 parts, among them U36 4081, U37 4081, U38 4081, U39 4069

Commit message: Add files via upload
Parts:
- U36, U37, U38, U39: footprint (none) -> Package_DIP:CERDIP-14_W7.62mm_SideBrazed_LongPads_Socket

Commit message: Add files via upload
Parts:
- renumbered U37 to U31, U36 to U32, U38 to U33, U39 to U34
Changed lines of the file:
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@@
 		(dnp no)
 		(fields_autoplaced yes)
-		(property "Reference" "U36"
+		(property "Reference" "U32"
 			(at 57.15 38.0916 90)
 			(effects
@@
 			(project ""
 				(path "/1bd2ca98-343e-4f04-8d6c-1f7257d9e9fe/60cf81cc-e4e5-4751-8bdc-8a094e4e39c9"
-					(reference "U36")
+					(reference "U32")
 					(unit 2)
 				)
@@
 		(dnp no)
 		(fields_autoplaced yes)
-		(property "Reference" "#PWR011"
+		(property "Reference" "#PWR019"
 			(at 201.93 36.83 0)
 			(effects
@@
 			(project "DTS"
 				(path "/1bd2ca98-343e-4f04-8d6c-1f7257d9e9fe/60cf81cc-e4e5-4751-8bdc-8a094e4e39c9"
-					(reference "#PWR011")
+					(reference "#PWR019")
 					(unit 1)
 				)
@@
 		(dnp no)
 		(fields_autoplaced yes)
-		(property "Reference" "U37"
+		(property "Reference" "U31"
 			(at 93.98 85.0816 90)
 			(effects
@@
 			(project ""
 				(path "/1bd2ca98-343e-4f04-8d6c-1f7257d9e9fe/60cf81cc-e4e5-4751-8bdc-8a094e4e39c9"
-					(reference "U37")
+					(reference "U31")
 					(unit 4)
 				)
@@
 		(dnp no)
 		(fields_autoplaced yes)
-		(property "Reference" "U37"
+		(property "Reference" "U31"
 			(at 55.88 102.87 90)
 			(effects
@@
 			(project ""
 				(path "/1bd2ca98-343e-4f04-8d6c-1f7257d9e9fe/60cf81cc-e4e5-4751-8bdc-8a094e4e39c9"
-					(reference "U37")
+					(reference "U31")
 					(unit 5)
 				)
@@
 		(dnp no)
 		(fields_autoplaced yes)
-		(property "Reference" "#PWR09"
+		(property "Reference" "#PWR017"
 			(at 124.46 36.83 0)
 			(effects
@@
 			(project "DTS"
 				(path "/1bd2ca98-343e-4f04-8d6c-1f7257d9e9fe/60cf81cc-e4e5-4751-8bdc-8a094e4e39c9"
-					(reference "#PWR09")
+					(reference "#PWR017")
 					(unit 1)
 				)
@@
 		(dnp no)
 		(fields_autoplaced yes)
-		(property "Reference" "#PWR010"
+		(property "Reference" "#PWR018"
 			(at 124.46 66.04 0)
 			(effects
@@
 			(project "DTS"
 				(path "/1bd2ca98-343e-4f04-8d6c-1f7257d9e9fe/60cf81cc-e4e5-4751-8bdc-8a094e4e39c9"
-					(reference "#PWR010")
+					(reference "#PWR018")
 					(unit 1)
 				)
@@
 		(dnp no)
 		(fields_autoplaced yes)
-		(property "Reference" "U38"
+		(property "Reference" "U33"
 			(at 96.52 135.8816 90)
 			(effects
@@
 			(project ""
 				(path "/1bd2ca98-343e-4f04-8d6c-1f7257d9e9fe/60cf81cc-e4e5-4751-8bdc-8a094e4e39c9"
-					(reference "U38")
+					(reference "U33")
 					(unit 4)
 				)
@@
 		(dnp no)
 		(fields_autoplaced yes)
-		(property "Reference" "U37"
+		(property "Reference" "U31"
 			(at 74.93 85.0816 90)
 			(effects
@@
 			(project ""
 				(path "/1bd2ca98-343e-4f04-8d6c-1f7257d9e9fe/60cf81cc-e4e5-4751-8bdc-8a094e4e39c9"
-					(reference "U37")
+					(reference "U31")
 					(unit 3)
 				)
@@
 		(dnp no)
 		(fields_autoplaced yes)
-		(property "Reference" "U39"
+		(property "Reference" "U34"
 			(at 161.29 135.8899 90)
 			(effects
@@
 			(project ""
 				(path "/1bd2ca98-343e-4f04-8d6c-1f7257d9e9fe/60cf81cc-e4e5-4751-8bdc-8a094e4e39c9"
-					(reference "U39")
+					(reference "U34")
 					(unit 2)
 				)
@@
 		(dnp no)
 		(fields_autoplaced yes)
-		(property "Reference" "U38"
+		(property "Reference" "U33"
 			(at 77.47 135.8816 90)
 			(effects
@@
 			(project ""
 				(path "/1bd2ca98-343e-4f04-8d6c-1f7257d9e9fe/60cf81cc-e4e5-4751-8bdc-8a094e4e39c9"
-					(reference "U38")
+					(reference "U33")
 					(unit 3)
 				)
@@
 		(dnp no)
 		(fields_autoplaced yes)
-		(property "Reference" "U39"
+		(property "Reference" "U34"
 			(at 191.77 135.8899 90)
 			(effects
@@
 			(project ""
 				(path "/1bd2ca98-343e-4f04-8d6c-1f7257d9e9fe/60cf81cc-e4e5-4751-8bdc-8a094e4e39c9"
-					(reference "U39")
+					(reference "U34")
 					(unit 4)
 				)
@@
 		(dnp no)
 		(fields_autoplaced yes)
-		(property "Reference" "U36"
+		(property "Reference" "U32"
 			(at 95.25 36.8216 90)
 			(effects
@@
 			(project ""
 				(path "/1bd2ca98-343e-4f04-8d6c-1f7257d9e9fe/60cf81cc-e4e5-4751-8bdc-8a094e4e39c9"
-					(reference "U36")
+					(reference "U32")
 					(unit 4)
 				)
@@
 		(dnp no)
 		(fields_autoplaced yes)
-		(property "Reference" "U39"
+		(property "Reference" "U34"
 			(at 223.52 135.8899 90)
 			(effects
@@
 			(project ""
 				(path "/1bd2ca98-343e-4f04-8d6c-1f7257d9e9fe/60cf81cc-e4e5-4751-8bdc-8a094e4e39c9"
-					(reference "U39")
+					(reference "U34")
 					(unit 6)
 				)
@@
 		(dnp no)
 		(fields_autoplaced yes)
-		(property "Reference" "U36"
+		(property "Reference" "U32"
 			(at 36.83 38.0916 90)
 			(effects
@@
 			(project ""
 				(path "/1bd2ca98-343e-4f04-8d6c-1f7257d9e9fe/60cf81cc-e4e5-4751-8bdc-8a094e4e39c9"
-					(reference "U36")
+					(reference "U32")
 					(unit 1)
 				)
@@
 		(dnp no)
 		(fields_autoplaced yes)
-		(property "Reference" "U39"
+		(property "Reference" "U34"
 			(at 181.61 146.05 90)
 			(effects
@@
 			(project ""
 				(path "/1bd2ca98-343e-4f04-8d6c-1f7257d9e9fe/60cf81cc-e4e5-4751-8bdc-8a094e4e39c9"
-					(reference "U39")
+					(reference "U34")
 					(unit 7)
 				)
@@
 		(dnp no)
 		(fields_autoplaced yes)
-		(property "Reference" "U39"
+		(property "Reference" "U34"
 			(at 176.53 135.8899 90)
 			(effects
@@
 			(project ""
 				(path "/1bd2ca98-343e-4f04-8d6c-1f7257d9e9fe/60cf81cc-e4e5-4751-8bdc-8a094e4e39c9"
-					(reference "U39")
+					(reference "U34")
 					(unit 3)
 				)
@@
 		(dnp no)
 		(fields_autoplaced yes)
-		(property "Reference" "U36"
+		(property "Reference" "U32"
 			(at 76.2 36.8216 90)
 			(effects
@@
 			(project ""
 				(path "/1bd2ca98-343e-4f04-8d6c-1f7257d9e9fe/60cf81cc-e4e5-4751-8bdc-8a094e4e39c9"
-					(reference "U36")
+					(reference "U32")
 					(unit 3)
 				)
@@
 		(dnp no)
 		(fields_autoplaced yes)
-		(property "Reference" "U37"
+		(property "Reference" "U31"
 			(at 55.88 86.3516 90)
 			(effects
@@
 			(project ""
 				(path "/1bd2ca98-343e-4f04-8d6c-1f7257d9e9fe/60cf81cc-e4e5-4751-8bdc-8a094e4e39c9"
-					(reference "U37")
+					(reference "U31")
 					(unit 2)
 				)
@@
 		(dnp no)
 		(fields_autoplaced yes)
-		(property "Reference" "U39"
+		(property "Reference" "U34"
 			(at 146.05 135.8899 90)
 			(effects
@@
 			(project ""
 				(path "/1bd2ca98-343e-4f04-8d6c-1f7257d9e9fe/60cf81cc-e4e5-4751-8bdc-8a094e4e39c9"
-					(reference "U39")
+					(reference "U34")
 					(unit 1)
 				)
@@
 		(dnp no)
 		(fields_autoplaced yes)
-		(property "Reference" "U38"
+		(property "Reference" "U33"
 			(at 59.69 152.4 90)
 			(effects
@@
 			(project ""
 				(path "/1bd2ca98-343e-4f04-8d6c-1f7257d9e9fe/60cf81cc-e4e5-4751-8bdc-8a094e4e39c9"
-					(reference "U38")
+					(reference "U33")
 					(unit 5)
 				)
@@
 		(dnp no)
 		(fields_autoplaced yes)
-		(property "Reference" "U36"
+		(property "Reference" "U32"
 			(at 57.15 54.61 90)
 			(effects
@@
 			(project ""
 				(path "/1bd2ca98-343e-4f04-8d6c-1f7257d9e9fe/60cf81cc-e4e5-4751-8bdc-8a094e4e39c9"
-					(reference "U36")
+					(reference "U32")
 					(unit 5)
 				)
@@
 		(dnp no)
 		(fields_autoplaced yes)
-		(property "Reference" "U38"
+		(property "Reference" "U33"
 			(at 58.42 135.8816 90)
 			(effects
@@
 			(project ""
 				(path "/1bd2ca98-343e-4f04-8d6c-1f7257d9e9fe/60cf81cc-e4e5-4751-8bdc-8a094e4e39c9"
-					(reference "U38")
+					(reference "U33")
 					(unit 2)
 				)
@@
 		(dnp no)
 		(fields_autoplaced yes)
-		(property "Reference" "U37"
+		(property "Reference" "U31"
 			(at 35.56 86.3516 90)
 			(effects
@@
 			(project ""
 				(path "/1bd2ca98-343e-4f04-8d6c-1f7257d9e9fe/60cf81cc-e4e5-4751-8bdc-8a094e4e39c9"
-					(reference "U37")
+					(reference "U31")
 					(unit 1)
 				)
@@
 		(dnp no)
 		(fields_autoplaced yes)
-		(property "Reference" "U39"
+		(property "Reference" "U34"
 			(at 207.01 135.8899 90)
 			(effects
@@
 			(project ""
 				(path "/1bd2ca98-343e-4f04-8d6c-1f7257d9e9fe/60cf81cc-e4e5-4751-8bdc-8a094e4e39c9"
-					(reference "U39")
+					(reference "U34")
 					(unit 5)
 				)
@@
 		(dnp no)
 		(fields_autoplaced yes)
-		(property "Reference" "U38"
+		(property "Reference" "U33"
 			(at 39.37 135.8816 90)
 			(effects
@@
 			(project ""
 				(path "/1bd2ca98-343e-4f04-8d6c-1f7257d9e9fe/60cf81cc-e4e5-4751-8bdc-8a094e4e39c9"
-					(reference "U38")
+					(reference "U33")
 					(unit 1)
 				)

Commit message: Add files via upload
Parts:
- removed U31, U32, U33: 4081, Package_DIP:CERDIP-14_W7.62mm_SideBrazed_LongPads_Socket, symbol 4xxx:4081
- removed U34: 4069, Package_DIP:CERDIP-14_W7.62mm_SideBrazed_LongPads_Socket, symbol 4xxx:4069
- added U12, U2, U7: 4081, Package_DIP:CERDIP-14_W7.62mm_SideBrazed_LongPads_Socket, symbol 4xxx:4081
- added U37: 4069, Package_DIP:CERDIP-14_W7.62mm_SideBrazed_LongPads_Socket, symbol 4xxx:4069
Connections:
- net (A0B2)': now also U37.10
- net (A1B2)': now also U37.8
- net (A2B0)': now also U37.6
- net (A2B1)': now also U37.4
- net A0: now also U2.9, U7.13
- net A0B1: now also U2.10
- net A0B2: now also U37.11, U7.11
- net A1: now also U2.6, U7.2, U7.9
- net A1B0: now also U2.4
- net A1B1: now also U7.3
- net A1B2: now also U37.9, U7.10
- net A2: now also U12.2, U7.6
- net A2B0: now also U37.5
- net A2B1: now also U12.3, U37.3
- net A2B2: now also U7.4
- net B0: now also U2.5
- net B1: now also U12.1, U2.8, U7.1
- net B2: now also U7.12, U7.5, U7.8
- net OUT0: now also U2.3
- net OUT5: now also U37.2
- net cout6: now also U37.1
- no-connect marks 0 -> 6
Other:
- sheet FullAdder: file FullAdder.kicad_sch -> fa4.kicad_sch
- sheet FullAdder ports: added none; removed GND, VCC
- sheet FullAdder1: file FullAdder.kicad_sch -> fa5.kicad_sch
- sheet FullAdder1 ports: added none; removed GND, VCC
- sheet FullAdder2: file FullAdder.kicad_sch -> fa6.kicad_sch
- sheet FullAdder2 ports: added none; removed GND, VCC
- sheet FullAdder3: file FullAdder.kicad_sch -> fa7.kicad_sch
- sheet FullAdder3 ports: added none; removed GND, VCC
- sheet FullAdder4: file FullAdder.kicad_sch -> fa8.kicad_sch
- sheet FullAdder4 ports: added none; removed GND, VCC
- sheet FullAdder5: file FullAdder.kicad_sch -> fa9.kicad_sch
- sheet FullAdder5 ports: added none; removed GND, VCC

Commit message: Add files via upload
Connections:
- net A0: now also U2.2
- net B0: now also U2.1
Changed lines of the file:
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@@
 	(hierarchical_label "B0"
 		(shape input)
-		(at 34.29 31.75 90)
+		(at 34.29 33.02 90)
 		(effects
 			(font
@@
 	(hierarchical_label "A0"
 		(shape input)
-		(at 29.21 31.75 90)
+		(at 29.21 33.02 90)
 		(effects
 			(font

Commit message: Add files via upload
Connections:
- net A2: now also U2.13
- net A2B0: now also U2.11
- net B0: now also U2.12
Changed lines of the file:
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@@
-	(wire
-		(pts
-			(xy 71.12 48.26) (xy 71.12 46.99)
-		)
-		(stroke
-			(width 0)
-			(type default)
-		)
-	)
 	(wire
 		(pts
@@
 	)
 	(label "A2B0"
-		(at 90.17 46.99 0)
+		(at 90.17 48.26 0)
 		(effects
 			(font
@@
 	)
 	(label "A0B1"
-		(at 71.12 46.99 0)
+		(at 71.12 48.26 0)
 		(effects
 			(font
@@
 	(hierarchical_label "B0"
 		(shape input)
-		(at 92.71 31.75 90)
+		(at 92.71 33.02 90)
 		(effects
 			(font
@@
 	(hierarchical_label "A2"
 		(shape input)
-		(at 87.63 31.75 90)
-		(effects
-			(font
+		(at 87.63 33.02 90)
+		(effects
+			(font
