File: multiplexer_3b.kicad_sch (KiCad schematic)
At the start: 4 parts, among them U13 4069, U14 4081, U15 4081, U16 4071

Commit message: Add files via upload
Parts:
- U13, U14, U15, U16: footprint (none) -> Package_DIP:CERDIP-14_W7.62mm_SideBrazed_LongPads_Socket

Commit message: Add files via upload
Parts:
- renumbered U13 to U15, U15 to U17, U14 to U18
Changed lines of the file:
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@@
 		(dnp no)
 		(fields_autoplaced yes)
-		(property "Reference" "U13"
+		(property "Reference" "U15"
 			(at 38.1 116.84 0)
 			(effects
@@
 			(project ""
 				(path "/1bd2ca98-343e-4f04-8d6c-1f7257d9e9fe/fcec0733-85ae-4916-ae1b-af5045bbbd48"
-					(reference "U13")
+					(reference "U15")
 					(unit 2)
 				)
@@
 		(dnp no)
 		(fields_autoplaced yes)
-		(property "Reference" "U13"
+		(property "Reference" "U15"
 			(at 38.1 130.81 0)
 			(effects
@@
 			(project ""
 				(path "/1bd2ca98-343e-4f04-8d6c-1f7257d9e9fe/fcec0733-85ae-4916-ae1b-af5045bbbd48"
-					(reference "U13")
+					(reference "U15")
 					(unit 3)
 				)
@@
 		(dnp no)
 		(fields_autoplaced yes)
-		(property "Reference" "U14"
+		(property "Reference" "U18"
 			(at 107.9417 54.61 0)
 			(effects
@@
 			(project ""
 				(path "/1bd2ca98-343e-4f04-8d6c-1f7257d9e9fe/fcec0733-85ae-4916-ae1b-af5045bbbd48"
-					(reference "U14")
+					(reference "U18")
 					(unit 2)
 				)
@@
 		(dnp no)
 		(fields_autoplaced yes)
-		(property "Reference" "U14"
+		(property "Reference" "U18"
 			(at 147.32 31.7499 0)
 			(effects
@@
 			(project ""
 				(path "/1bd2ca98-343e-4f04-8d6c-1f7257d9e9fe/fcec0733-85ae-4916-ae1b-af5045bbbd48"
-					(reference "U14")
+					(reference "U18")
 					(unit 5)
 				)
@@
 		(dnp no)
 		(fields_autoplaced yes)
-		(property "Reference" "U15"
+		(property "Reference" "U17"
 			(at 170.18 31.7499 0)
 			(effects
@@
 			(project ""
 				(path "/1bd2ca98-343e-4f04-8d6c-1f7257d9e9fe/fcec0733-85ae-4916-ae1b-af5045bbbd48"
-					(reference "U15")
+					(reference "U17")
 					(unit 5)
 				)
@@
 		(dnp no)
 		(fields_autoplaced yes)
-		(property "Reference" "U14"
+		(property "Reference" "U18"
 			(at 107.9417 73.66 0)
 			(effects
@@
 			(project ""
 				(path "/1bd2ca98-343e-4f04-8d6c-1f7257d9e9fe/fcec0733-85ae-4916-ae1b-af5045bbbd48"
-					(reference "U14")
+					(reference "U18")
 					(unit 3)
 				)
@@
 		(dnp no)
 		(fields_autoplaced yes)
-		(property "Reference" "U15"
+		(property "Reference" "U17"
 			(at 140.9617 54.61 0)
 			(effects
@@
 			(project ""
 				(path "/1bd2ca98-343e-4f04-8d6c-1f7257d9e9fe/fcec0733-85ae-4916-ae1b-af5045bbbd48"
-					(reference "U15")
+					(reference "U17")
 					(unit 1)
 				)
@@
 		(dnp no)
 		(fields_autoplaced yes)
-		(property "Reference" "U15"
+		(property "Reference" "U17"
 			(at 69.8417 116.84 0)
 			(effects
@@
 			(project ""
 				(path "/1bd2ca98-343e-4f04-8d6c-1f7257d9e9fe/fcec0733-85ae-4916-ae1b-af5045bbbd48"
-					(reference "U15")
+					(reference "U17")
 					(unit 3)
 				)
@@
 		(dnp no)
 		(fields_autoplaced yes)
-		(property "Reference" "U13"
+		(property "Reference" "U15"
 			(at 40.64 33.02 0)
 			(effects
@@
 			(project ""
 				(path "/1bd2ca98-343e-4f04-8d6c-1f7257d9e9fe/fcec0733-85ae-4916-ae1b-af5045bbbd48"
-					(reference "U13")
+					(reference "U15")
 					(unit 1)
 				)
@@
 		(dnp no)
 		(fields_autoplaced yes)
-		(property "Reference" "U13"
+		(property "Reference" "U15"
 			(at 80.01 31.7499 0)
 			(effects
@@
 			(project ""
 				(path "/1bd2ca98-343e-4f04-8d6c-1f7257d9e9fe/fcec0733-85ae-4916-ae1b-af5045bbbd48"
-					(reference "U13")
+					(reference "U15")
 					(unit 7)
 				)
@@
 		(dnp no)
 		(fields_autoplaced yes)
-		(property "Reference" "U13"
+		(property "Reference" "U15"
 			(at 38.1 146.05 0)
 			(effects
@@
 			(project ""
 				(path "/1bd2ca98-343e-4f04-8d6c-1f7257d9e9fe/fcec0733-85ae-4916-ae1b-af5045bbbd48"
-					(reference "U13")
+					(reference "U15")
 					(unit 4)
 				)
@@
 		(dnp no)
 		(fields_autoplaced yes)
-		(property "Reference" "U15"
+		(property "Reference" "U17"
 			(at 140.9617 72.39 0)
 			(effects
@@
 			(project ""
 				(path "/1bd2ca98-343e-4f04-8d6c-1f7257d9e9fe/fcec0733-85ae-4916-ae1b-af5045bbbd48"
-					(reference "U15")
+					(reference "U17")
 					(unit 2)
 				)
@@
 		(dnp no)
 		(fields_autoplaced yes)
-		(property "Reference" "U14"
+		(property "Reference" "U18"
 			(at 107.9417 36.83 0)
 			(effects
@@
 			(project ""
 				(path "/1bd2ca98-343e-4f04-8d6c-1f7257d9e9fe/fcec0733-85ae-4916-ae1b-af5045bbbd48"
-					(reference "U14")
+					(reference "U18")
 					(unit 1)
 				)
@@
 		(dnp no)
 		(fields_autoplaced yes)
-		(property "Reference" "U13"
+		(property "Reference" "U15"
 			(at 38.1 161.29 0)
 			(effects
@@
 			(project ""
 				(path "/1bd2ca98-343e-4f04-8d6c-1f7257d9e9fe/fcec0733-85ae-4916-ae1b-af5045bbbd48"
-					(reference "U13")
+					(reference "U15")
 					(unit 5)
 				)
@@
 		(dnp no)
 		(fields_autoplaced yes)
-		(property "Reference" "U14"
+		(property "Reference" "U18"
 			(at 107.9417 91.44 0)
 			(effects
@@
 			(project ""
 				(path "/1bd2ca98-343e-4f04-8d6c-1f7257d9e9fe/fcec0733-85ae-4916-ae1b-af5045bbbd48"
-					(reference "U14")
+					(reference "U18")
 					(unit 4)
 				)
@@
 		(dnp no)
 		(fields_autoplaced yes)
-		(property "Reference" "U13"
+		(property "Reference" "U15"
 			(at 38.1 176.53 0)
 			(effects
@@
 			(project ""
 				(path "/1bd2ca98-343e-4f04-8d6c-1f7257d9e9fe/fcec0733-85ae-4916-ae1b-af5045bbbd48"
-					(reference "U13")
+					(reference "U15")
 					(unit 6)
 				)
@@
 		(dnp no)
 		(fields_autoplaced yes)
-		(property "Reference" "U15"
+		(property "Reference" "U17"
 			(at 69.8417 130.81 0)
 			(effects
@@
 			(project ""
 				(path "/1bd2ca98-343e-4f04-8d6c-1f7257d9e9fe/fcec0733-85ae-4916-ae1b-af5045bbbd48"
-					(reference "U15")
+					(reference "U17")
 					(unit 4)
 				)
