File: multiplexer_6b.kicad_sch (KiCad schematic)
At the start: 6 parts, among them U17 4069, U18 4071, U19 4081, U20 4081, U21 4071, U22 4081

Commit message: Add files via upload
Parts:
- U17, U18, U19, U20, U21, U22: footprint (none) -> Package_DIP:CERDIP-14_W7.62mm_SideBrazed_LongPads_Socket

Commit message: Add files via upload
Parts:
- removed U17: 4069, Package_DIP:CERDIP-14_W7.62mm_SideBrazed_LongPads_Socket, symbol 4xxx:4069
- added U19: 4069, Package_DIP:CERDIP-14_W7.62mm_SideBrazed_LongPads_Socket, symbol 4xxx:4069
- renumbered U18 to U20, U20 to U22, U19 to U23, U22 to U24
Connections:
- net (ctrl)': now also U19.2
- net GND: now also U19.7 (VSS)
- net VCC: now also U19.14 (VDD)
- net ctrl: now also U19.1
