File: Signed_Extended.kicad_sch (KiCad schematic)
At the start: 7 parts, among them U1 4081, U10 4071, U18 4069, U27 4069, U46 4071, U48 4081, U6 4081

Commit message: Add files via upload
Parts:
- removed U1, U48, U6: 4081, Package_DIP:CERDIP-14_W7.62mm_SideBrazed_LongPads_Socket, symbol 4xxx:4081
- removed U10, U46: 4071, Package_DIP:CERDIP-14_W7.62mm_SideBrazed_LongPads_Socket, symbol 4xxx:4071
- removed U18, U27: 4069, Package_DIP:CERDIP-14_W7.62mm_SideBrazed_LongPads_Socket, symbol 4xxx:4069
- added U59: 4069, Package_DIP:CERDIP-14_W7.62mm_SideBrazed_LongPads_Socket, symbol 4xxx:4069
- added U60, U61, U63: 4081, Package_DIP:CERDIP-14_W7.62mm_SideBrazed_LongPads_Socket, symbol 4xxx:4081
- added U62: 4071, Package_DIP:CERDIP-14_W7.62mm_SideBrazed_LongPads_Socket, symbol 4xxx:4071
Connections:
- net (A2^B2)': now also U59.12, U63.1
- net (c^(A2^B2))': now also U62.10, U63.8
- net A2: now also U59.3, U61.2, U61.9
- net A2': now also U59.4, U61.13, U61.5
- net A2'B2: now also U61.4, U62.1
- net A2'S2: now also U61.11, U62.5
- net A2B2': now also U61.3, U62.2
- net A2S2': now also U61.10, U62.6
- net A2^B2: now also U59.13, U62.3, U63.5
- net A2^S2: now also U62.4, U63.9
- net B2: now also U59.1, U61.6
- net B2': now also U59.2, U61.1
- net S2: now also U59.5, U61.12, U63.12
- net S2': now also U59.6, U60.2, U61.8
- net c: now also U59.11, U63.6
- net c': now also U59.10, U63.2
- net c'(A2^B2)': now also U62.9, U63.3
- net c(A2^B2): now also U62.8, U63.4
- net overflow: now also U59.9, U60.1, U63.10
- net overflow': now also U59.8, U63.13
- net overflow'S2: now also U62.13, U63.11
- net overflowS2': now also U60.3, U62.12
- net signed: now also U62.11
- new net GND: U59.14 (VDD), U60.14 (VDD), U61.14 (VDD), U62.14 (VDD), U63.14 (VDD)
- new net VCC: U59.7 (VSS), U60.7 (VSS), U61.7 (VSS), U62.7 (VSS), U63.7 (VSS)
