File: Signed_Extended.kicad_sch (KiCad schematic)
At the start: 5 parts, among them U40 4081, U65 4071, U66 4069, U67 4081, U68 4081

Commit message: Add files via upload
Parts:
- U40, U65, U66, U67, U68: footprint (none) -> Package_DIP:CERDIP-14_W7.62mm_SideBrazed_LongPads_Socket

Commit message: Add files via upload
Parts:
- renumbered U66 to U59, U68 to U60, U40 to U61, U65 to U62, U67 to U63
Changed lines of the file:
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@@
 		(dnp no)
 		(fields_autoplaced yes)
-		(property "Reference" "U68"
+		(property "Reference" "U60"
 			(at 29.21 177.7916 90)
 			(effects
@@
 			(project ""
 				(path "/1bd2ca98-343e-4f04-8d6c-1f7257d9e9fe/6b755f33-010e-4b1b-a5fd-e02d322a419a"
-					(reference "U68")
+					(reference "U60")
 					(unit 2)
 				)
@@
 		(dnp no)
 		(fields_autoplaced yes)
-		(property "Reference" "U66"
+		(property "Reference" "U59"
 			(at 60.96 91.4399 90)
 			(effects
@@
 			(project ""
 				(path "/1bd2ca98-343e-4f04-8d6c-1f7257d9e9fe/6b755f33-010e-4b1b-a5fd-e02d322a419a"
-					(reference "U66")
+					(reference "U59")
 					(unit 4)
 				)
@@
 		(dnp no)
 		(fields_autoplaced yes)
-		(property "Reference" "U66"
+		(property "Reference" "U59"
 			(at 27.94 69.8499 90)
 			(effects
@@
 			(project ""
 				(path "/1bd2ca98-343e-4f04-8d6c-1f7257d9e9fe/6b755f33-010e-4b1b-a5fd-e02d322a419a"
-					(reference "U66")
+					(reference "U59")
 					(unit 1)
 				)
@@
 		(dnp no)
 		(fields_autoplaced yes)
-		(property "Reference" "U40"
+		(property "Reference" "U61"
 			(at 223.52 96.52 90)
 			(effects
@@
 			(project ""
 				(path "/1bd2ca98-343e-4f04-8d6c-1f7257d9e9fe/6b755f33-010e-4b1b-a5fd-e02d322a419a"
-					(reference "U40")
+					(reference "U61")
 					(unit 5)
 				)
@@
 		(dnp no)
 		(fields_autoplaced yes)
-		(property "Reference" "U66"
+		(property "Reference" "U59"
 			(at 223.52 115.57 90)
 			(effects
@@
 			(project ""
 				(path "/1bd2ca98-343e-4f04-8d6c-1f7257d9e9fe/6b755f33-010e-4b1b-a5fd-e02d322a419a"
-					(reference "U66")
+					(reference "U59")
 					(unit 7)
 				)
@@
 		(dnp no)
 		(fields_autoplaced yes)
-		(property "Reference" "U67"
+		(property "Reference" "U63"
 			(at 132.08 83.8116 90)
 			(effects
@@
 			(project ""
 				(path "/1bd2ca98-343e-4f04-8d6c-1f7257d9e9fe/6b755f33-010e-4b1b-a5fd-e02d322a419a"
-					(reference "U67")
+					(reference "U63")
 					(unit 1)
 				)
@@
 		(dnp no)
 		(fields_autoplaced yes)
-		(property "Reference" "U40"
+		(property "Reference" "U61"
 			(at 99.06 43.1716 90)
 			(effects
@@
 			(project ""
 				(path "/1bd2ca98-343e-4f04-8d6c-1f7257d9e9fe/6b755f33-010e-4b1b-a5fd-e02d322a419a"
-					(reference "U40")
+					(reference "U61")
 					(unit 4)
 				)
@@
 		(dnp no)
 		(fields_autoplaced yes)
-		(property "Reference" "U66"
+		(property "Reference" "U59"
 			(at 60.96 69.8499 90)
 			(effects
@@
 			(project ""
 				(path "/1bd2ca98-343e-4f04-8d6c-1f7257d9e9fe/6b755f33-010e-4b1b-a5fd-e02d322a419a"
-					(reference "U66")
+					(reference "U59")
 					(unit 3)
 				)
@@
 		(dnp no)
 		(fields_autoplaced yes)
-		(property "Reference" "U65"
+		(property "Reference" "U62"
 			(at 130.81 43.1799 90)
 			(effects
@@
 			(project ""
 				(path "/1bd2ca98-343e-4f04-8d6c-1f7257d9e9fe/6b755f33-010e-4b1b-a5fd-e02d322a419a"
-					(reference "U65")
+					(reference "U62")
 					(unit 1)
 				)
@@
 		(dnp no)
 		(fields_autoplaced yes)
-		(property "Reference" "U68"
+		(property "Reference" "U60"
 			(at 134.62 115.5616 90)
 			(effects
@@
 			(project ""
 				(path "/1bd2ca98-343e-4f04-8d6c-1f7257d9e9fe/6b755f33-010e-4b1b-a5fd-e02d322a419a"
-					(reference "U68")
+					(reference "U60")
 					(unit 1)
 				)
@@
 		(dnp no)
 		(fields_autoplaced yes)
-		(property "Reference" "U66"
+		(property "Reference" "U59"
 			(at 44.45 91.4399 90)
 			(effects
@@
 			(project ""
 				(path "/1bd2ca98-343e-4f04-8d6c-1f7257d9e9fe/6b755f33-010e-4b1b-a5fd-e02d322a419a"
-					(reference "U66")
+					(reference "U59")
 					(unit 6)
 				)
@@
 		(dnp no)
 		(fields_autoplaced yes)
-		(property "Reference" "U67"
+		(property "Reference" "U63"
 			(at 189.23 83.8116 90)
 			(effects
@@
 			(project ""
 				(path "/1bd2ca98-343e-4f04-8d6c-1f7257d9e9fe/6b755f33-010e-4b1b-a5fd-e02d322a419a"
-					(reference "U67")
+					(reference "U63")
 					(unit 4)
 				)
@@
 		(dnp no)
 		(fields_autoplaced yes)
-		(property "Reference" "U68"
+		(property "Reference" "U60"
 			(at 223.52 60.96 90)
 			(effects
@@
 			(project ""
 				(path "/1bd2ca98-343e-4f04-8d6c-1f7257d9e9fe/6b755f33-010e-4b1b-a5fd-e02d322a419a"
-					(reference "U68")
+					(reference "U60")
 					(unit 5)
 				)
@@
 		(dnp no)
 		(fields_autoplaced yes)
-		(property "Reference" "U67"
+		(property "Reference" "U63"
 			(at 168.91 83.8116 90)
 			(effects
@@
 			(project ""
 				(path "/1bd2ca98-343e-4f04-8d6c-1f7257d9e9fe/6b755f33-010e-4b1b-a5fd-e02d322a419a"
-					(reference "U67")
+					(reference "U63")
 					(unit 3)
 				)
@@
 		(dnp no)
 		(fields_autoplaced yes)
-		(property "Reference" "U68"
+		(property "Reference" "U60"
 			(at 46.99 177.7916 90)
 			(effects
@@
 			(project ""
 				(path "/1bd2ca98-343e-4f04-8d6c-1f7257d9e9fe/6b755f33-010e-4b1b-a5fd-e02d322a419a"
-					(reference "U68")
+					(reference "U60")
 					(unit 3)
 				)
@@
 		(dnp no)
 		(fields_autoplaced yes)
-		(property "Reference" "U65"
+		(property "Reference" "U62"
 			(at 186.69 43.1799 90)
 			(effects
@@
 			(project ""
 				(path "/1bd2ca98-343e-4f04-8d6c-1f7257d9e9fe/6b755f33-010e-4b1b-a5fd-e02d322a419a"
-					(reference "U65")
+					(reference "U62")
 					(unit 4)
 				)
@@
 		(dnp no)
 		(fields_autoplaced yes)
-		(property "Reference" "U40"
+		(property "Reference" "U61"
 			(at 80.01 43.1716 90)
 			(effects
@@
 			(project ""
 				(path "/1bd2ca98-343e-4f04-8d6c-1f7257d9e9fe/6b755f33-010e-4b1b-a5fd-e02d322a419a"
-					(reference "U40")
+					(reference "U61")
 					(unit 3)
 				)
@@
 		(dnp no)
 		(fields_autoplaced yes)
-		(property "Reference" "U67"
+		(property "Reference" "U63"
 			(at 223.52 80.01 90)
 			(effects
@@
 			(project ""
 				(path "/1bd2ca98-343e-4f04-8d6c-1f7257d9e9fe/6b755f33-010e-4b1b-a5fd-e02d322a419a"
-					(reference "U67")
+					(reference "U63")
 					(unit 5)
 				)
@@
 		(dnp no)
 		(fields_autoplaced yes)
-		(property "Reference" "U40"
+		(property "Reference" "U61"
 			(at 62.23 43.1716 90)
 			(effects
@@
 			(project ""
 				(path "/1bd2ca98-343e-4f04-8d6c-1f7257d9e9fe/6b755f33-010e-4b1b-a5fd-e02d322a419a"
-					(reference "U40")
+					(reference "U61")
 					(unit 2)
 				)
@@
 		(dnp no)
 		(fields_autoplaced yes)
-		(property "Reference" "U65"
+		(property "Reference" "U62"
 			(at 167.64 43.1799 90)
 			(effects
@@
 			(project ""
 				(path "/1bd2ca98-343e-4f04-8d6c-1f7257d9e9fe/6b755f33-010e-4b1b-a5fd-e02d322a419a"
-					(reference "U65")
+					(reference "U62")
 					(unit 3)
 				)
@@
 		(dnp no)
 		(fields_autoplaced yes)
-		(property "Reference" "U66"
+		(property "Reference" "U59"
 			(at 27.94 91.4399 90)
 			(effects
@@
 			(project ""
 				(path "/1bd2ca98-343e-4f04-8d6c-1f7257d9e9fe/6b755f33-010e-4b1b-a5fd-e02d322a419a"
-					(reference "U66")
+					(reference "U59")
 					(unit 5)
 				)
@@
 		(dnp no)
 		(fields_autoplaced yes)
-		(property "Reference" "U65"
+		(property "Reference" "U62"
 			(at 223.52 134.62 90)
 			(effects
@@
 			(project ""
 				(path "/1bd2ca98-343e-4f04-8d6c-1f7257d9e9fe/6b755f33-010e-4b1b-a5fd-e02d322a419a"
-					(reference "U65")
+					(reference "U62")
 					(unit 5)
 				)
@@
 		(dnp no)
 		(fields_autoplaced yes)
-		(property "Reference" "U40"
+		(property "Reference" "U61"
 			(at 43.18 43.1716 90)
 			(effects
@@
 			(project ""
 				(path "/1bd2ca98-343e-4f04-8d6c-1f7257d9e9fe/6b755f33-010e-4b1b-a5fd-e02d322a419a"
-					(reference "U40")
+					(reference "U61")
 					(unit 1)
 				)
@@
 		(dnp no)
 		(fields_autoplaced yes)
-		(property "Reference" "U66"
+		(property "Reference" "U59"
 			(at 44.45 69.8499 90)
 			(effects
@@
 			(project ""
 				(path "/1bd2ca98-343e-4f04-8d6c-1f7257d9e9fe/6b755f33-010e-4b1b-a5fd-e02d322a419a"
-					(reference "U66")
+					(reference "U59")
 					(unit 2)
 				)
@@
 		(dnp no)
 		(fields_autoplaced yes)
-		(property "Reference" "U68"
+		(property "Reference" "U60"
 			(at 64.77 177.7916 90)
 			(effects
@@
 			(project ""
 				(path "/1bd2ca98-343e-4f04-8d6c-1f7257d9e9fe/6b755f33-010e-4b1b-a5fd-e02d322a419a"
-					(reference "U68")
+					(reference "U60")
 					(unit 4)
 				)
@@
 		(dnp no)
 		(fields_autoplaced yes)
-		(property "Reference" "U65"
+		(property "Reference" "U62"
 			(at 148.59 43.1799 90)
 			(effects
@@
 			(project ""
 				(path "/1bd2ca98-343e-4f04-8d6c-1f7257d9e9fe/6b755f33-010e-4b1b-a5fd-e02d322a419a"
-					(reference "U65")
+					(reference "U62")
 					(unit 2)
 				)
@@
 		(dnp no)
 		(fields_autoplaced yes)
-		(property "Reference" "U67"
+		(property "Reference" "U63"
 			(at 149.86 83.8116 90)
 			(effects
@@
 			(project ""
 				(path "/1bd2ca98-343e-4f04-8d6c-1f7257d9e9fe/6b755f33-010e-4b1b-a5fd-e02d322a419a"
-					(reference "U67")
+					(reference "U63")
 					(unit 2)
 				)

Commit message: Add files via upload
Parts:
- removed U59: 4069, Package_DIP:CERDIP-14_W7.62mm_SideBrazed_LongPads_Socket, symbol 4xxx:4069
- removed U60, U61, U63: 4081, Package_DIP:CERDIP-14_W7.62mm_SideBrazed_LongPads_Socket, symbol 4xxx:4081
- removed U62: 4071, Package_DIP:CERDIP-14_W7.62mm_SideBrazed_LongPads_Socket, symbol 4xxx:4071
- added U1, U48, U6: 4081, Package_DIP:CERDIP-14_W7.62mm_SideBrazed_LongPads_Socket, symbol 4xxx:4081
- added U10, U46: 4071, Package_DIP:CERDIP-14_W7.62mm_SideBrazed_LongPads_Socket, symbol 4xxx:4071
- added U18, U27: 4069, Package_DIP:CERDIP-14_W7.62mm_SideBrazed_LongPads_Socket, symbol 4xxx:4069
Connections:
- net (A2^B2)': now also U1.5, U27.6
- net (c^(A2^B2))': now also U1.12, U10.3
- net A2: now also U18.13, U48.13, U48.6
- net A2': now also U1.2, U18.12, U48.8
- net A2'B2: now also U46.12, U48.10
- net A2'S2: now also U1.3, U46.8
- net A2B2': now also U46.13, U48.4
- net A2S2': now also U46.9, U48.11
- net A2^B2: now also U1.8, U27.5, U46.11
- net A2^S2: now also U1.13, U46.10
- net B2: now also U18.11, U48.9
- net B2': now also U18.10, U48.5
- net S2: now also U1.1, U27.1, U6.1
- net S2': now also U27.2, U48.12, U6.6
- net c: now also U1.9, U27.3
- net c': now also U1.6, U27.4
- net c'(A2^B2)': now also U1.4, U10.2
- net c(A2^B2): now also U1.10, U10.1
- net overflow: now also U1.11, U27.9, U6.5
- net overflow': now also U27.8, U6.2
- net overflow'S2: now also U10.6, U6.3
- net overflowS2': now also U10.5, U6.4
- net signed: now also U10.4
