File: fa4.kicad_sch (KiCad schematic)
At the start: 4 parts, among them U35 4081, U36 4069, U37 4071, U38 4081

Commit message: Add files via upload
Parts:
- removed U35, U38: 4081, Package_DIP:CERDIP-14_W7.62mm_SideBrazed_LongPads_Socket, symbol 4xxx:4081
- removed U36: 4069, Package_DIP:CERDIP-14_W7.62mm_SideBrazed_LongPads_Socket, symbol 4xxx:4069
- removed U37: 4071, Package_DIP:CERDIP-14_W7.62mm_SideBrazed_LongPads_Socket, symbol 4xxx:4071
- added U12, U16: 4081, Package_DIP:CERDIP-14_W7.62mm_SideBrazed_LongPads_Socket, symbol 4xxx:4081
- added U14, U37: 4069, Package_DIP:CERDIP-14_W7.62mm_SideBrazed_LongPads_Socket, symbol 4xxx:4069
- added U31: 4071, Package_DIP:CERDIP-14_W7.62mm_SideBrazed_LongPads_Socket, symbol 4xxx:4071
Connections:
- net (xy' + x'y)': now also U14.6, U16.8
- net c_in: now also U14.3, U16.13, U16.9
- net c_in': now also U14.4, U16.6
- net c_out: now also U31.10
- net sum: now also U31.4
- net temp1: now also U16.4, U31.5
- net temp2: now also U16.10, U31.6
- net temp3: now also U16.11, U31.9
- net x: now also U12.5, U12.8, U37.13
- net x': now also U12.13, U37.12
- net x'y: now also U31.2
- net xor_out: now also U14.5, U16.12, U16.5, U31.3
- net xy: now also U12.4, U31.8
- net xy': now also U12.10, U12.11, U31.1
- net y: now also U12.12, U12.6, U14.1
- net y': now also U12.9, U14.2

Commit message: Add files via upload
Connections:
- net x'y: now also U12.11
- net xy': no longer U12.11
Changed lines of the file:
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@@
+		)
+	)
+	(label "x'y"
+		(at 157.48 57.15 0)
+		(effects
+			(font
+				(size 1.27 1.27)
+			)
+			(justify left bottom)
 		)
 	)
@@
 		(effects
 			(font
-				(size 1.27 1.27)
-			)
-			(justify left bottom)
-		)
-	)
-	(label "xy'"
-		(at 157.48 57.15 0)
-		(effects
-			(font
