File: fa4.kicad_sch (KiCad schematic)
At the start: 5 parts, among them U12 4081, U14 4069, U16 4081, U31 4071, U37 4069

Commit message: Add files via upload
Connections:
- net x'y: now also U12.11
- net xy': no longer U12.11
