File: fa8.kicad_sch (KiCad schematic)
At the start: 4 parts, among them U51 4081, U52 4069, U53 4071, U54 4081

Commit message: Add files via upload
Parts:
- removed U51, U54: 4081, Package_DIP:CERDIP-14_W7.62mm_SideBrazed_LongPads_Socket, symbol 4xxx:4081
- removed U52: 4069, Package_DIP:CERDIP-14_W7.62mm_SideBrazed_LongPads_Socket, symbol 4xxx:4069
- removed U53: 4071, Package_DIP:CERDIP-14_W7.62mm_SideBrazed_LongPads_Socket, symbol 4xxx:4071
- added U32, U5: 4069, Package_DIP:CERDIP-14_W7.62mm_SideBrazed_LongPads_Socket, symbol 4xxx:4069
- added U39, U42: 4081, Package_DIP:CERDIP-14_W7.62mm_SideBrazed_LongPads_Socket, symbol 4xxx:4081
- added U43: 4071, Package_DIP:CERDIP-14_W7.62mm_SideBrazed_LongPads_Socket, symbol 4xxx:4071
Connections:
- net (xy' + x'y)': now also U42.8, U5.2
- net c_in: now also U32.13, U42.13, U42.9
- net c_in': now also U32.12, U42.6
- net c_out: now also U43.10
- net sum: now also U43.4
- net temp1: now also U42.4, U43.5
- net temp2: now also U42.10, U43.6
- net temp3: now also U42.11, U43.9
- net x: now also U32.9, U39.5, U39.8
- net x': now also U32.8, U39.13
- net x'y: now also U43.2
- net xor_out: now also U42.12, U42.5, U43.3, U5.1
- net xy: now also U39.4, U43.8
- net xy': now also U39.10, U39.11, U43.1
- net y: now also U32.11, U39.12, U39.6
- net y': now also U32.10, U39.9

Commit message: Add files via upload
Connections:
- net x'y: now also U39.11
- net xy': no longer U39.11
Changed lines of the file:
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@@
-	)
-	(label "xy'"
-		(at 157.48 57.15 0)
-		(effects
-			(font
-				(size 1.27 1.27)
-			)
-			(justify left bottom)
-		)
 	)
 	(label "xy'"
@@
 		(effects
 			(font
+				(size 1.27 1.27)
+			)
+			(justify left bottom)
+		)
+	)
+	(label "x'y"
+		(at 157.48 57.15 0)
+		(effects
+			(font
