File: fa8.kicad_sch (KiCad schematic)
At the start: 5 parts, among them U32 4069, U39 4081, U42 4081, U43 4071, U5 4069

Commit message: Add files via upload
Connections:
- net x'y: now also U39.11
- net xy': no longer U39.11
