File: mux3b.kicad_sch (KiCad schematic)
At the start: 4 parts, among them U15 4069, U16 4071, U17 4081, U18 4081

Commit message: Add files via upload
Parts:
- removed U15: 4069, Package_DIP:CERDIP-14_W7.62mm_SideBrazed_LongPads_Socket, symbol 4xxx:4069
- removed U16: 4071, Package_DIP:CERDIP-14_W7.62mm_SideBrazed_LongPads_Socket, symbol 4xxx:4071
- removed U17, U18: 4081, Package_DIP:CERDIP-14_W7.62mm_SideBrazed_LongPads_Socket, symbol 4xxx:4081
- added U29, U34: 4081, Package_DIP:CERDIP-14_W7.62mm_SideBrazed_LongPads_Socket, symbol 4xxx:4081
- added U3: 4071, Package_DIP:CERDIP-14_W7.62mm_SideBrazed_LongPads_Socket, symbol 4xxx:4071
- added U4: 4069, Package_DIP:CERDIP-14_W7.62mm_SideBrazed_LongPads_Socket, symbol 4xxx:4069
Connections:
- net (ctrl)': now also U34.13, U34.2, U34.9, U4.8
- net ctrl: now also U29.13, U29.9, U34.6, U4.9
- net i0_0: now also U34.8
- net i0_1: now also U34.12
- net i0_2: now also U34.1
- net i1_0: now also U34.5
- net i1_1: now also U29.8
- net i1_2: now also U29.12
- net iout_0: now also U3.3
- net iout_1: now also U3.4
- net iout_2: now also U3.10
- net temp1: now also U3.1, U34.10
- net temp2: now also U3.5, U34.11
- net temp3: now also U3.8, U34.3
- net temp4: now also U3.2, U34.4
- net temp5: now also U29.10, U3.6
- net temp6: now also U29.11, U3.9
