File: mux6b1.kicad_sch (KiCad schematic)
At the start: 6 parts, among them U19 4069, U20 4071, U21 4071, U22 4081, U23 4081, U24 4081

Commit message: Add files via upload
Parts:
- removed U19: 4069, Package_DIP:CERDIP-14_W7.62mm_SideBrazed_LongPads_Socket, symbol 4xxx:4069
- removed U20: 4071, Package_DIP:CERDIP-14_W7.62mm_SideBrazed_LongPads_Socket, symbol 4xxx:4071
- removed unit 3 of U21
- removed unit 4 of U21
- removed unit 5 of U21
- removed U22, U23, U24: 4081, Package_DIP:CERDIP-14_W7.62mm_SideBrazed_LongPads_Socket, symbol 4xxx:4081
- added U17: 4071, Package_DIP:CERDIP-14_W7.62mm_SideBrazed_LongPads_Socket, symbol 4xxx:4071
- added U27: 4069, Package_DIP:CERDIP-14_W7.62mm_SideBrazed_LongPads_Socket, symbol 4xxx:4069
- added U38, U41, U44: 4081, Package_DIP:CERDIP-14_W7.62mm_SideBrazed_LongPads_Socket, symbol 4xxx:4081
Connections:
- net (ctrl)': now also U27.10, U38.2, U38.6, U38.9, U41.13, U41.9, U44.2
- net ctrl: now also U27.11, U38.13, U41.2, U41.6, U44.13, U44.6, U44.9
- net i0_0: now also U38.1
- net i0_1: now also U38.5
- net i0_2: now also U38.8
- net i0_3: now also U41.8
- net i0_4: now also U41.12
- net i0_5: now also U44.1
- net i1_0: now also U38.12
- net i1_1: now also U41.1
- net i1_2: now also U41.5
- net i1_3: now also U44.5
- net i1_4: now also U44.8
- net i1_5: now also U44.12
- net iout_0: now also U17.3
- net iout_1: now also U17.4
- net iout_2: now also U17.10
- net iout_3: now also U17.11
- net temp1: now also U17.1, U38.3
- net temp10: now also U17.13, U44.4
- net temp11: now also U44.10
- net temp12: now also U44.11
- net temp2: now also U17.5, U38.4
- net temp3: now also U17.8, U38.10
- net temp4: now also U17.2, U38.11
- net temp5: now also U17.6, U41.3
- net temp6: now also U17.9, U41.4
- net temp7: now also U17.12, U41.10
- net temp8: now also U41.11
- net temp9: now also U44.3
