File: mux6b2.kicad_sch (KiCad schematic)
At the start: 6 parts, among them U25 4069, U26 4071, U27 4071, U28 4081, U29 4081, U30 4081

Commit message: Add files via upload
Parts:
- removed U25: 4069, Package_DIP:CERDIP-14_W7.62mm_SideBrazed_LongPads_Socket, symbol 4xxx:4069
- removed unit 5 of U26
- removed U27: 4071, Package_DIP:CERDIP-14_W7.62mm_SideBrazed_LongPads_Socket, symbol 4xxx:4071
- removed unit 5 of U28
- removed U29, U30: 4081, Package_DIP:CERDIP-14_W7.62mm_SideBrazed_LongPads_Socket, symbol 4xxx:4081
- added U21: 4071, Package_DIP:CERDIP-14_W7.62mm_SideBrazed_LongPads_Socket, symbol 4xxx:4071
- added U23, U47: 4081, Package_DIP:CERDIP-14_W7.62mm_SideBrazed_LongPads_Socket, symbol 4xxx:4081
- added U27: 4069, Package_DIP:CERDIP-14_W7.62mm_SideBrazed_LongPads_Socket, symbol 4xxx:4069
Connections:
- net (ctrl)': now also U23.13, U23.9, U27.12, U47.2, U47.6, U47.9; no longer U28.6, U28.9
- net ctrl: now also U28.6, U28.9, U23.2, U23.6, U27.13, U47.13
- net i0_0: now also U47.1; no longer U28.1
- net i0_1: now also U47.5; no longer U28.5
- net i0_2: now also U47.8; no longer U28.8
- net i0_3: now also U23.8
- net i0_4: now also U23.12
- net i0_5: now also U28.1
- net i1_0: now also U47.12; no longer U28.12
- net i1_1: now also U23.1
- net i1_2: now also U23.5
- net i1_3: now also U28.5
- net i1_4: now also U28.8
- net i1_5: now also U28.12
- net iout_0: now also U21.10; no longer U26.3
- net iout_1: now also U21.11; no longer U26.4
- net iout_2: now also U26.3; no longer U26.10
- net iout_3: now also U26.4; no longer U26.11
- net iout_4: now also U26.10
- net iout_5: now also U26.11
- net temp1: now also U21.8, U47.3; no longer U26.1, U28.3
- net temp10: now also U26.6, U28.4; no longer U26.13
- net temp11: now also U26.9, U28.10
- net temp12: now also U26.13, U28.11
- net temp2: now also U21.12, U47.4; no longer U26.5, U28.4
- net temp3: now also U26.1, U47.10; no longer U26.8, U28.10
- net temp4: now also U21.9, U47.11; no longer U26.2, U28.11
- net temp5: now also U21.13, U23.3; no longer U26.6
- net temp6: now also U26.2, U23.4; no longer U26.9
- net temp7: now also U26.5, U23.10; no longer U26.12
- net temp8: now also U26.8, U23.11
- net temp9: now also U26.12, U28.3
