File: fa2.kicad_sch (KiCad schematic)
At the start: 4 parts, among them U10 4081, U7 4081, U8 4069, U9 4071

Commit message: Add files via upload
Parts:
- removed U10, U7: 4081, Package_DIP:CERDIP-14_W7.62mm_SideBrazed_LongPads_Socket, symbol 4xxx:4081
- removed U8: 4069, Package_DIP:CERDIP-14_W7.62mm_SideBrazed_LongPads_Socket, symbol 4xxx:4069
- removed U9: 4071, Package_DIP:CERDIP-14_W7.62mm_SideBrazed_LongPads_Socket, symbol 4xxx:4071
- added U13, U8: 4071, Package_DIP:CERDIP-14_W7.62mm_SideBrazed_LongPads_Socket, symbol 4xxx:4071
- added U15, U19: 4081, Package_DIP:CERDIP-14_W7.62mm_SideBrazed_LongPads_Socket, symbol 4xxx:4081
- added U9: 4069, Package_DIP:CERDIP-14_W7.62mm_SideBrazed_LongPads_Socket, symbol 4xxx:4069
Connections:
- net (xy' + x'y)': now also U19.8, U9.12
- net c_in: now also U19.13, U19.9, U9.11
- net c_in': now also U19.6, U9.10
- net c_out: now also U13.3
- net sum: now also U8.11
- net temp1: now also U19.4, U8.12
- net temp2: now also U19.10, U8.13
- net temp3: now also U13.2, U19.11
- net x: now also U15.12, U15.8, U9.5
- net x': now also U19.2, U9.6
- net x'y: now also U8.9
- net xor_out: now also U19.12, U19.5, U8.10, U9.13
- net xy: now also U13.1, U15.10
- net xy': now also U15.11, U19.3, U8.8
- net y: now also U15.9, U19.1, U9.9
- net y': now also U15.13, U9.8
