File: fa2.kicad_sch (KiCad schematic)
At the start: 5 parts, among them U13 4071, U15 4081, U19 4081, U8 4071, U9 4069

Commit message: Add files via upload
Connections:
- net temp2: no longer U19.10
- net x'y: now also U19.3
- net xy': no longer U19.3
