File: fa5.kicad_sch (KiCad schematic)
At the start: 4 parts, among them U39 4081, U40 4069, U41 4071, U42 4081

Commit message: Add files via upload
Parts:
- removed U39, U42: 4081, Package_DIP:CERDIP-14_W7.62mm_SideBrazed_LongPads_Socket, symbol 4xxx:4081
- removed U40: 4069, Package_DIP:CERDIP-14_W7.62mm_SideBrazed_LongPads_Socket, symbol 4xxx:4069
- removed U41: 4071, Package_DIP:CERDIP-14_W7.62mm_SideBrazed_LongPads_Socket, symbol 4xxx:4071
- added U14, U22: 4069, Package_DIP:CERDIP-14_W7.62mm_SideBrazed_LongPads_Socket, symbol 4xxx:4069
- added U16, U20, U25: 4081, Package_DIP:CERDIP-14_W7.62mm_SideBrazed_LongPads_Socket, symbol 4xxx:4081
- added U31, U36: 4071, Package_DIP:CERDIP-14_W7.62mm_SideBrazed_LongPads_Socket, symbol 4xxx:4071
Connections:
- net (xy' + x'y)': now also U14.12, U20.12
- net c_in: now also U14.11, U20.13, U25.2
- net c_in': now also U14.10, U20.9
- net c_out: now also U31.11
- net sum: now also U36.4
- net temp1: now also U20.10, U36.5
- net temp2: now also U20.11, U36.6
- net temp3: now also U25.3, U31.13
- net x: now also U16.1, U20.1, U22.1
- net x': now also U20.6, U22.2
- net x'y: now also U36.2
- net xor_out: now also U14.13, U20.8, U25.1, U36.3
- net xy: now also U16.3, U31.12
- net xy': now also U20.3, U20.4, U36.1
- net y: now also U14.9, U16.2, U20.5
- net y': now also U14.8, U20.2
