File: fa5.kicad_sch (KiCad schematic)
At the start: 7 parts, among them U1 4081, U10 4071, U18 4069, U27 4069, U46 4071, U48 4081, U6 4081

Commit message: Add files via upload
Parts:
- removed U1, U48, U6: 4081, Package_DIP:CERDIP-14_W7.62mm_SideBrazed_LongPads_Socket, symbol 4xxx:4081
- removed U10, U46: 4071, Package_DIP:CERDIP-14_W7.62mm_SideBrazed_LongPads_Socket, symbol 4xxx:4071
- removed U18, U27: 4069, Package_DIP:CERDIP-14_W7.62mm_SideBrazed_LongPads_Socket, symbol 4xxx:4069
- added U14, U22: 4069, Package_DIP:CERDIP-14_W7.62mm_SideBrazed_LongPads_Socket, symbol 4xxx:4069
- added U16, U20, U25: 4081, Package_DIP:CERDIP-14_W7.62mm_SideBrazed_LongPads_Socket, symbol 4xxx:4081
- added U31, U36: 4071, Package_DIP:CERDIP-14_W7.62mm_SideBrazed_LongPads_Socket, symbol 4xxx:4071
Connections:
- new net (xy' + x'y)': U14.12, U20.12
- new net c_in: U14.11, U20.13, U25.2
- new net c_in': U14.10, U20.9
- new net c_out: U31.11
- new net sum: U36.4
- new net temp1: U20.10, U36.5
- new net temp2: U20.11, U36.6
- new net temp3: U25.3, U31.13
- new net x: U16.1, U20.1, U22.1
- new net x': U20.6, U22.2
- new net x'y: U36.2
- new net xor_out: U14.13, U20.8, U25.1, U36.3
- new net xy: U16.3, U31.12
- new net xy': U20.3, U20.4, U36.1
- new net y: U14.9, U16.2, U20.5
- new net y': U14.8, U20.2

Commit message: Add files via upload
Connections:
- net x'y: now also U20.4
- net xy': no longer U20.4
Changed lines of the file:
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@@
-		)
-	)
-	(label "xy'"
-		(at 157.48 57.15 0)
-		(effects
-			(font
-				(size 1.27 1.27)
-			)
-			(justify left bottom)
 		)
 	)
@@
 		(effects
 			(font
+				(size 1.27 1.27)
+			)
+			(justify left bottom)
+		)
+	)
+	(label "x'y"
+		(at 157.48 57.15 0)
+		(effects
+			(font
