File: fa5.kicad_sch (KiCad schematic)
At the start: 7 parts, among them U14 4069, U16 4081, U20 4081, U22 4069, U25 4081, U31 4071, U36 4071

Commit message: Add files via upload
Connections:
- net x'y: now also U20.4
- net xy': no longer U20.4
