File: fa7.kicad_sch (KiCad schematic)
At the start: 4 parts, among them U47 4081, U48 4069, U49 4071, U50 4081

Commit message: Add files via upload
Parts:
- removed U47, U50: 4081, Package_DIP:CERDIP-14_W7.62mm_SideBrazed_LongPads_Socket, symbol 4xxx:4081
- removed U48: 4069, Package_DIP:CERDIP-14_W7.62mm_SideBrazed_LongPads_Socket, symbol 4xxx:4069
- removed U49: 4071, Package_DIP:CERDIP-14_W7.62mm_SideBrazed_LongPads_Socket, symbol 4xxx:4071
- added U22, U32: 4069, Package_DIP:CERDIP-14_W7.62mm_SideBrazed_LongPads_Socket, symbol 4xxx:4069
- added U30, U35, U39: 4081, Package_DIP:CERDIP-14_W7.62mm_SideBrazed_LongPads_Socket, symbol 4xxx:4081
- added U40: 4071, Package_DIP:CERDIP-14_W7.62mm_SideBrazed_LongPads_Socket, symbol 4xxx:4071
Connections:
- net (xy' + x'y)': now also U32.6, U35.12
- net c_in: now also U32.3, U35.13, U39.2
- net c_in': now also U32.4, U35.9
- net c_out: now also U40.11
- net sum: now also U40.10
- net temp1: now also U35.10, U40.8
- net temp2: now also U35.11, U40.9
- net temp3: now also U39.3, U40.13
- net x: now also U22.13, U30.1, U35.1
- net x': now also U22.12, U35.6
- net x'y: now also U40.6
- net xor_out: now also U32.5, U35.8, U39.1, U40.4
- net xy: now also U30.3, U40.12
- net xy': now also U35.3, U35.4, U40.5
- net y: now also U30.2, U32.1, U35.5
- net y': now also U32.2, U35.2
