File: fa7.kicad_sch (KiCad schematic)
At the start: 6 parts, among them U22 4069, U30 4081, U32 4069, U35 4081, U39 4081, U40 4071

Commit message: Add files via upload
Connections:
- net x'y: now also U35.4
- net xy': no longer U35.4
