File: fa7.kicad_sch (KiCad schematic)
At the start: 7 parts, among them U1 4081, U10 4071, U18 4069, U27 4069, U46 4071, U48 4081, U6 4081

Commit message: Add files via upload
Parts:
- removed U1, U48, U6: 4081, Package_DIP:CERDIP-14_W7.62mm_SideBrazed_LongPads_Socket, symbol 4xxx:4081
- removed U10, U46: 4071, Package_DIP:CERDIP-14_W7.62mm_SideBrazed_LongPads_Socket, symbol 4xxx:4071
- removed U18, U27: 4069, Package_DIP:CERDIP-14_W7.62mm_SideBrazed_LongPads_Socket, symbol 4xxx:4069
- added U22, U32: 4069, Package_DIP:CERDIP-14_W7.62mm_SideBrazed_LongPads_Socket, symbol 4xxx:4069
- added U30, U35, U39: 4081, Package_DIP:CERDIP-14_W7.62mm_SideBrazed_LongPads_Socket, symbol 4xxx:4081
- added U40: 4071, Package_DIP:CERDIP-14_W7.62mm_SideBrazed_LongPads_Socket, symbol 4xxx:4071
Connections:
- new net (xy' + x'y)': U32.6, U35.12
- new net c_in: U32.3, U35.13, U39.2
- new net c_in': U32.4, U35.9
- new net c_out: U40.11
- new net sum: U40.10
- new net temp1: U35.10, U40.8
- new net temp2: U35.11, U40.9
- new net temp3: U39.3, U40.13
- new net x: U22.13, U30.1, U35.1
- new net x': U22.12, U35.6
- new net x'y: U40.6
- new net xor_out: U32.5, U35.8, U39.1, U40.4
- new net xy: U30.3, U40.12
- new net xy': U35.3, U35.4, U40.5
- new net y: U30.2, U32.1, U35.5
- new net y': U32.2, U35.2

Commit message: Add files via upload
Connections:
- net x'y: now also U35.4
- net xy': no longer U35.4
Changed lines of the file:
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@@
+		)
+	)
+	(label "x'y"
+		(at 157.3631 57.15 0)
+		(effects
+			(font
+				(size 1.27 1.27)
+			)
+			(justify left bottom)
 		)
 	)
@@
 		(effects
 			(font
-				(size 1.27 1.27)
-			)
-			(justify left bottom)
-		)
-	)
-	(label "xy'"
-		(at 157.48 57.15 0)
-		(effects
-			(font

Commit message: Add files via upload
Changed lines of the file:
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@@
 	(wire
 		(pts
-			(xy 152.4 57.15) (xy 157.48 57.15)
+			(xy 152.4 57.15) (xy 158.75 57.15)
 		)
 		(stroke
@@
 	)
 	(label "x'y"
-		(at 157.3631 57.15 0)
-		(effects
-			(font
+		(at 158.75 57.15 0)
+		(effects
+			(font
