File: DTS.kicad_pcb (KiCad board)
At the start: 2 copper layers, 160 x 156.5 mm, 55 parts, among them J1 Conn_01x02_Pin, J2 Conn_01x06_Pin, J3 Conn_01x02_Pin, J4 Conn_01x06_Pin, SW1 SW_DIP_x01, U1 4081, U10 4071, U11 4081, U12 4081, U13 4071, U14 4069, U15 4081, U16 4081, U17 4071, U18 4069, U19 4081, U2 4081, U20 4081, U21 4071, U22 4069, U23 4081, U24 4081, U25 4081, U26 4071, U27 4069, U28 4081, U29 4081, U3 4071, U30 4081, U31 4071, U32 4069, U34 4081, U35 4081, U36 4071, U37 4069, U38 4081, U39 4081, U4 4069, U40 4071, U41 4081, U42 4081, U43 4071, U44 4081, U45 4081, U46 4071, U47 4081, U48 4081, U49 LM7805_TO220, U5 4069, U6 4081, U7 4081, U8 4071, U9 4069

Commit message: Add files via upload
Parts:
- added D1: LED, Connector_PinHeader_2.54mm:PinHeader_1x02_P2.54mm_Vertical, F.Cu at (224.8, 114.8)
- added D10: LED, Connector_PinHeader_2.54mm:PinHeader_1x02_P2.54mm_Vertical, F.Cu at (229.4, 121.9)
- added D11: LED, Connector_PinHeader_2.54mm:PinHeader_1x02_P2.54mm_Vertical, F.Cu at (234.0, 121.9)
- added D12: LED, Connector_PinHeader_2.54mm:PinHeader_1x02_P2.54mm_Vertical, F.Cu at (238.6, 121.9)
- added D13: LED, Connector_PinHeader_2.54mm:PinHeader_1x02_P2.54mm_Vertical, F.Cu at (243.2, 121.9)
- added D14: LED, Connector_PinHeader_2.54mm:PinHeader_1x02_P2.54mm_Vertical, F.Cu at (247.7, 121.9)
- added D15: LED, Connector_PinHeader_2.54mm:PinHeader_1x02_P2.54mm_Vertical, F.Cu at (252.3, 121.9)
- added D2: LED, Connector_PinHeader_2.54mm:PinHeader_1x02_P2.54mm_Vertical, F.Cu at (229.4, 114.8)
- added D3: LED, Connector_PinHeader_2.54mm:PinHeader_1x02_P2.54mm_Vertical, F.Cu at (234.0, 114.8)
- added D4: LED, Connector_PinHeader_2.54mm:PinHeader_1x02_P2.54mm_Vertical, F.Cu at (238.6, 114.8)
- added D5: LED, Connector_PinHeader_2.54mm:PinHeader_1x02_P2.54mm_Vertical, F.Cu at (243.2, 114.8)
- added D6: LED, Connector_PinHeader_2.54mm:PinHeader_1x02_P2.54mm_Vertical, F.Cu at (247.7, 114.8)
- added D7: LED, Connector_PinHeader_2.54mm:PinHeader_1x02_P2.54mm_Vertical, F.Cu at (252.3, 114.8)
- added D8: LED, Connector_PinHeader_2.54mm:PinHeader_1x02_P2.54mm_Vertical, F.Cu at (256.9, 114.8)
- added D9: LED, Connector_PinHeader_2.54mm:PinHeader_1x02_P2.54mm_Vertical, F.Cu at (224.8, 121.9)
- added R1: R, Connector_PinHeader_2.54mm:PinHeader_1x02_P2.54mm_Vertical, F.Cu at (256.9, 121.9)
- added R10: R, Connector_PinHeader_2.54mm:PinHeader_1x02_P2.54mm_Vertical, F.Cu at (224.8, 136.2)
- added R11: R, Connector_PinHeader_2.54mm:PinHeader_1x02_P2.54mm_Vertical, F.Cu at (229.4, 136.2)
- added R12: R, Connector_PinHeader_2.54mm:PinHeader_1x02_P2.54mm_Vertical, F.Cu at (234.0, 136.2)
- added R13: R, Connector_PinHeader_2.54mm:PinHeader_1x02_P2.54mm_Vertical, F.Cu at (238.6, 136.2)
- added R14: R, Connector_PinHeader_2.54mm:PinHeader_1x02_P2.54mm_Vertical, F.Cu at (243.2, 136.2)
- added R2: R, Connector_PinHeader_2.54mm:PinHeader_1x02_P2.54mm_Vertical, F.Cu at (224.8, 129.1)
- added R3: R, Connector_PinHeader_2.54mm:PinHeader_1x02_P2.54mm_Vertical, F.Cu at (229.4, 129.1)
- added R4: R, Connector_PinHeader_2.54mm:PinHeader_1x02_P2.54mm_Vertical, F.Cu at (234.0, 129.1)
- added R5: R, Connector_PinHeader_2.54mm:PinHeader_1x02_P2.54mm_Vertical, F.Cu at (238.6, 129.1)
- added R6: R, Connector_PinHeader_2.54mm:PinHeader_1x02_P2.54mm_Vertical, F.Cu at (243.2, 129.1)
- added R7: R, Connector_PinHeader_2.54mm:PinHeader_1x02_P2.54mm_Vertical, F.Cu at (247.7, 129.1)
- added R8: R, Connector_PinHeader_2.54mm:PinHeader_1x02_P2.54mm_Vertical, F.Cu at (252.3, 129.1)
- added R9: R, Connector_PinHeader_2.54mm:PinHeader_1x02_P2.54mm_Vertical, F.Cu at (256.9, 129.1)
- added SW2: SW_DIP_x01, Connector_PinHeader_2.54mm:PinHeader_1x03_P2.54mm_Vertical, F.Cu at (224.8, 143.4)
- added SW3: SW_DIP_x01, Connector_PinHeader_2.54mm:PinHeader_1x03_P2.54mm_Vertical, F.Cu at (229.4, 143.4)
- added SW4: SW_DIP_x01, Connector_PinHeader_2.54mm:PinHeader_1x03_P2.54mm_Vertical, F.Cu at (234.0, 143.4)
- added SW5: SW_DIP_x01, Connector_PinHeader_2.54mm:PinHeader_1x03_P2.54mm_Vertical, F.Cu at (238.6, 143.4)
- added SW6: SW_DIP_x01, Connector_PinHeader_2.54mm:PinHeader_1x03_P2.54mm_Vertical, F.Cu at (243.2, 143.4)
- added SW7: SW_DIP_x01, Connector_PinHeader_2.54mm:PinHeader_1x03_P2.54mm_Vertical, F.Cu at (247.7, 143.4)
- added SW8: SW_DIP_x01, Connector_PinHeader_2.54mm:PinHeader_1x03_P2.54mm_Vertical, F.Cu at (252.3, 143.4)
- added SW9: SW_DIP_x01, Connector_PinHeader_2.54mm:PinHeader_1x03_P2.54mm_Vertical, F.Cu at (256.9, 143.4)
- C1, C2: footprint Capacitor_THT:C_Rect_L7.0mm_W2.0mm_P5.00mm -> Capacitor_THT:C_Radial_D6.3mm_H5.0mm_P2.50mm
- SW1: footprint Connector_PinSocket_2.54mm:PinSocket_1x02_P2.54mm_Vertical -> Connector_PinHeader_2.54mm:PinHeader_1x03_P2.54mm_Vertical
- moved U49 184.1 mm to (212.3, 47.1), turned to 180 degrees
- moved J1 176.4 mm to (210.6, 64.6), turned to 90 degrees
- moved C2 175.8 mm to (207.3, 42.1)
- moved SW1 169.7 mm to (210.3, 59.6), turned to 180 degrees
- moved C1 169.0 mm to (209.3, 52.6)
- moved U21 140.3 mm to (186.0, 54.7), turned to 90 degrees
- moved U11 119.7 mm to (160.8, 110.5), turned to 90 degrees
- moved U4 119.2 mm to (161.1, 137.0), turned to 90 degrees
- moved U3 117.2 mm to (160.8, 123.1), turned to 90 degrees
- moved U44 115.2 mm to (161.5, 54.7), turned to 90 degrees
- moved U15 112.6 mm to (184.3, 136.6), turned to 90 degrees
- moved J4 110.1 mm to (164.4, 145.8), turned to 90 degrees
- moved U42 106.4 mm to (111.1, 41.7), turned to 90 degrees
- moved U32 103.0 mm to (161.1, 82.7), turned to 90 degrees
- moved U10 102.4 mm to (65.1, 94.7), turned to 90 degrees
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Connections:
- net /Multiplexer_6b1/i0_0 renamed /mult0
- net /Multiplexer_6b1/i0_1 renamed /mult1
- net /Multiplexer_6b1/i0_2 renamed /mult2
- net /Multiplexer_6b1/i0_3 renamed /mult3
- net /Multiplexer_6b1/i0_4 renamed /mult4
- net /Multiplexer_6b1/i0_5 renamed /mult5
- net /Multiplexer_6b2/iout_0 renamed /output 0
- net /Multiplexer_6b2/iout_1 renamed /output 1
- net /Multiplexer_6b2/iout_2 renamed /output 2
- net /Multiplexer_6b2/iout_3 renamed /output 3
- net /Multiplexer_6b2/iout_4 renamed /output 4
- net /Multiplexer_6b2/iout_5 renamed /output 5
- J2 pad 1: x1 -> x0
- J2 pad 2: x2 -> x1
- J2 pad 3: x3 -> x2
- J2 pad 4: y1 -> y0
- J2 pad 5: y2 -> y1
- J2 pad 6: y3 -> y2
- U1 pad 1: s3 -> s2
- U11 pad 1: x1 -> x0
- U11 pad 12: xor1 -> xor0
- U11 pad 2: /y_signed1 -> /y_signed0
- U11 pad 5: x1 -> x0
- U11 pad 8: /y_signed1 -> /y_signed0
- U12 pad 1: y2 -> y1
- U12 pad 2: x3 -> x2
- U13 pad 10: s3 -> s2
- U13 pad 4: xor3 -> xor2
- U15 pad 12: x2 -> x1
- U15 pad 5: xor1 -> xor0
- U15 pad 8: x2 -> x1
- U15 pad 9: /y_signed2 -> /y_signed1
- U18 pad 1: x3 -> x2
- U18 pad 11: y3 -> y2
- U18 pad 13: x3 -> x2
- U18 pad 3: /y_signed3 -> /y_signed2
- U18 pad 9: xor3 -> xor2
- U19 pad 1: /y_signed2 -> /y_signed1
- U19 pad 12: xor2 -> xor1
- U19 pad 5: xor2 -> xor1
- U2 pad 5: y1 -> y0
- U2 pad 6: x2 -> x1
- U2 pad 8: y2 -> y1
- U2 pad 9: x1 -> x0
- U24 pad 1: x3 -> x2
- U24 pad 12: xor3 -> xor2
- U24 pad 2: /y_signed3 -> /y_signed2
- U24 pad 5: x3 -> x2
- U24 pad 8: /y_signed3 -> /y_signed2
- U27 pad 1: s3 -> s2
- U29 pad 12: /y3' -> /y2'
- U29 pad 5: xor3 -> xor2
- U29 pad 8: /y2' -> /y1'
- U3 pad 10: /y_signed3 -> /y_signed2
- U3 pad 3: /y_signed1 -> /y_signed0
- U3 pad 4: /y_signed2 -> /y_signed1
- U34 pad 1: y3 -> y2
- U34 pad 12: y2 -> y1
- U34 pad 5: /y1' -> /y0'
- U34 pad 8: y1 -> y0
- U38 pad 12: xor1 -> xor0
- U4 pad 11: x1 -> x0
- U4 pad 13: /y_signed1 -> /y_signed0
- U4 pad 5: y3 -> y0
- U4 pad 6: /y3' -> /y0'
- U41 pad 1: xor2 -> xor1
- U41 pad 5: xor3 -> xor2
- U44 pad 12: xor3 -> xor2
- U44 pad 5: xor3 -> xor2
- U44 pad 8: xor3 -> xor2
- U47 pad 1: s1 -> s0
- U47 pad 5: s2 -> s1
- U47 pad 8: s3 -> s2
- U48 pad 13: x3 -> x2
- U48 pad 6: x3 -> x2
- U48 pad 9: y3 -> y2
- U6 pad 1: s3 -> s2
- U7 pad 1: y2 -> y1
- U7 pad 12: y3 -> y2
- U7 pad 13: x1 -> x0
- U7 pad 2: x2 -> x1
- U7 pad 5: y3 -> y2
- U7 pad 6: x3 -> x2
- U7 pad 8: y3 -> y2
- U7 pad 9: x2 -> x1
- U8 pad 10: xor2 -> xor1
- U8 pad 11: s2 -> s1
- U8 pad 3: xor1 -> xor0
- U8 pad 4: s1 -> s0
- U9 pad 13: xor2 -> xor1
- U9 pad 3: xor1 -> xor0
- U9 pad 5: x2 -> x1
- U9 pad 9: /y_signed2 -> /y_signed1
Routing:
- net GND: track 0.00 -> 857.9 mm
- net VCC: track 0.00 -> 801.2 mm, vias 0 -> 1
- net ctrl_out0: track 0.00 -> 403.9 mm, vias 0 -> 6
- net y2: track 0.00 -> 380.5 mm, vias 0 -> 4
- net xor2: track 0.00 -> 233.8 mm, vias 0 -> 4
- net /Multiplier/(A1B2)': track 0.00 -> 212.7 mm, vias 0 -> 3
- net ctrl_out1: track 0.00 -> 204.7 mm, vias 0 -> 1
- net x2: track 0.00 -> 196.3 mm, vias 0 -> 1
- net x1: track 0.00 -> 184.0 mm
- net /Multiplier/(A0B2)': track 0.00 -> 178.1 mm, vias 0 -> 8
- net /Multiplier/cout3: track 0.00 -> 173.3 mm
- net /mult5: track 0.00 -> 164.0 mm, vias 0 -> 3
- net s2: track 0.00 -> 151.5 mm, vias 0 -> 3
- net /Multiplier/A2B2: track 0.00 -> 146.2 mm, vias 0 -> 1
- net x0: track 0.00 -> 141.6 mm
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Other:
- board size 160 x 156.5 mm -> 162.7 x 122 mm
- board text added: "ctr0"
- board text added: "ctr1"
- board text added: "io1"
- board text added: "io2"
- board text added: "io3"
- board text added: "io4"
- board text added: "io5"
- board text added: "io6"
- board text added: "x1"
- board text added: "x2"
- board text added: "x3"
- board text added: "y1"
- board text added: "y2"
- board text added: "y3"

Commit message: Add files via upload
Connections:
- U4 pad 1: y1 -> y0
- U4 pad 2: /y1' -> /y0'
- U4 pad 3: y2 -> y1
- U4 pad 4: /y2' -> /y1'
- U4 pad 5: y0 -> y2
- U4 pad 6: /y0' -> /y2'
Routing:
- net y2: track 380.5 -> 260.7 mm, vias 4 -> 3
- net y0: track 0.00 -> 96.1 mm, vias 0 -> 1
- net /y2': track 86.6 -> 52.0 mm, vias 2 -> 1
- net y1: track 96.1 -> 119.8 mm
- net /y0': track 0.00 -> 19.9 mm
- net /y1': track 19.9 -> 34.6 mm, vias 0 -> 1

Commit message: Add files via upload
Parts:
- moved D8 197.4 mm to (67.0, 61.0)
- moved R1 194.9 mm to (67.0, 78.0)
- moved R7 189.4 mm to (71.0, 61.0)
- moved SW9 189.1 mm to (87.0, 60.5)
- moved SW8 188.5 mm to (83.0, 60.5)
- moved R8 185.3 mm to (79.0, 63.5), turned to 180 degrees
- moved D7 178.9 mm to (76.0, 84.5)
- moved D6 178.8 mm to (71.5, 85.0)
- moved D5 178.7 mm to (67.0, 85.0)
- moved SW7 171.3 mm to (85.0, 90.0)
- moved R6 171.0 mm to (76.0, 93.0)
- moved R5 170.9 mm to (71.5, 93.0)
- moved R4 170.9 mm to (67.0, 92.7)
- moved SW6 170.2 mm to (85.0, 80.5)
- moved SW5 170.0 mm to (85.0, 70.5)
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Routing:
- net GND: track 857.9 -> 0.00 mm
- net VCC: track 801.2 -> 0.00 mm, vias 1 -> 0
- net ctrl_out0: track 403.9 -> 0.00 mm, vias 6 -> 0
- net y2: track 260.7 -> 0.00 mm, vias 3 -> 0
- net xor2: track 233.8 -> 0.00 mm, vias 4 -> 0
- net /Multiplier/(A1B2)': track 212.7 -> 0.00 mm, vias 3 -> 0
- net ctrl_out1: track 204.7 -> 0.00 mm, vias 1 -> 0
- net x2: track 196.3 -> 0.00 mm, vias 1 -> 0
- net x1: track 184.0 -> 0.00 mm
- net /Multiplier/(A0B2)': track 178.1 -> 0.00 mm, vias 8 -> 0
- net /Multiplier/cout3: track 173.3 -> 0.00 mm
- net /mult5: track 164.0 -> 0.00 mm, vias 3 -> 0
- net s2: track 151.5 -> 0.00 mm, vias 3 -> 0
- net /Multiplier/A2B2: track 146.2 -> 0.00 mm, vias 1 -> 0
- net x0: track 141.6 -> 0.00 mm
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Other:
- board text removed: "ctr0"
- board text removed: "ctr1"
- board text removed: "io1"
- board text removed: "io2"
- board text removed: "io3"
- board text removed: "io4"
- board text removed: "io5"
- board text removed: "io6"
- board text removed: "x1"
- board text removed: "x2"
- board text removed: "x3"
- board text removed: "y1"
- board text removed: "y2"
- board text removed: "y3"
