File: DTS.kicad_sch (KiCad schematic)
At the start: 9 parts, among them J4 Conn_01x06_Pin, J5 Conn_01x02_Pin, J6 Conn_01x02_Pin, J7 Conn_01x06_Pin, SW1 SW_DIP_x01, U23 4069, U69 LM7805_TO220

Commit message: Add files via upload
Parts:
- C1, C2: footprint (none) -> Capacitor_THT:C_Rect_L7.0mm_W2.0mm_P5.00mm
- J4, J7: footprint (none) -> Connector_PinHeader_2.54mm:PinHeader_1x06_P2.54mm_Vertical
- J5, J6: footprint (none) -> Connector_PinHeader_2.54mm:PinHeader_1x02_P2.54mm_Vertical
- SW1: footprint (none) -> Connector_PinSocket_2.54mm:PinSocket_1x02_P2.54mm_Vertical
- U23: footprint (none) -> Package_DIP:CERDIP-14_W7.62mm_SideBrazed_LongPads_Socket

Commit message: Add files via upload
Parts:
- renumbered J5 to J1, J4 to J2, J6 to J3, J7 to J4, U23 to U1, U69 to U2
Other:
- removed sheet Multiplexer_6b

Commit message: Add files via upload
Parts:
- removed U1: 4069, Package_DIP:CERDIP-14_W7.62mm_SideBrazed_LongPads_Socket, symbol 4xxx:4069
- added U1, U11, U12, U15, U16, U19, U2, U20, U23, U24, U25, U28, U29, U30, U34, U35, U38, U39, U41, U42, U44, U45, U47, U48, U6, U7: 4081, Package_DIP:CERDIP-14_W7.62mm_SideBrazed_LongPads_Socket, symbol 4xxx:4081
- added U10, U13, U17, U21, U26, U3, U31, U36, U40, U43, U46, U8: 4071, Package_DIP:CERDIP-14_W7.62mm_SideBrazed_LongPads_Socket, symbol 4xxx:4071
- added U14, U18, U22, U27, U32, U37, U4, U5, U9: 4069, Package_DIP:CERDIP-14_W7.62mm_SideBrazed_LongPads_Socket, symbol 4xxx:4069
- renumbered U2 to U49
Connections:
- net GND: now also U1.7 (VSS), U10.7 (VSS), U11.7 (VSS), U12.7 (VSS), U13.7 (VSS), U14.7 (VSS), U15.7 (VSS), U16.7 (VSS), U17.7 (VSS), U18.7 (VSS), U19.7 (VSS), U2.7 (VSS), U20.7 (VSS), U21.7 (VSS), U22.7 (VSS), U23.7 (VSS), U24.7 (VSS), U25.7 (VSS), U26.7 (VSS), U27.7 (VSS), U28.7 (VSS), U29.7 (VSS), U3.7 (VSS), U30.7 (VSS), U31.7 (VSS), U32.7 (VSS), U34.7 (VSS), U35.7 (VSS), U36.7 (VSS), U37.7 (VSS), U38.7 (VSS), U39.7 (VSS), U4.7 (VSS), U40.7 (VSS), U41.7 (VSS), U42.7 (VSS), U43.7 (VSS), U44.7 (VSS), U45.7 (VSS), U46.7 (VSS), U47.7 (VSS), U48.7 (VSS), U5.7 (VSS), U6.7 (VSS), U7.7 (VSS), U8.7 (VSS), U9.7 (VSS)
- net VCC: now also U1.14 (VDD), U10.14 (VDD), U11.14 (VDD), U12.14 (VDD), U13.14 (VDD), U14.14 (VDD), U15.14 (VDD), U16.14 (VDD), U17.14 (VDD), U18.14 (VDD), U19.14 (VDD), U2.14 (VDD), U20.14 (VDD), U21.14 (VDD), U22.14 (VDD), U23.14 (VDD), U24.14 (VDD), U25.14 (VDD), U26.14 (VDD), U27.14 (VDD), U28.14 (VDD), U29.14 (VDD), U3.14 (VDD), U30.14 (VDD), U31.14 (VDD), U32.14 (VDD), U34.14 (VDD), U35.14 (VDD), U36.14 (VDD), U37.14 (VDD), U38.14 (VDD), U39.14 (VDD), U4.14 (VDD), U40.14 (VDD), U41.14 (VDD), U42.14 (VDD), U43.14 (VDD), U44.14 (VDD), U45.14 (VDD), U46.14 (VDD), U47.14 (VDD), U48.14 (VDD), U5.14 (VDD), U6.14 (VDD), U7.14 (VDD), U8.14 (VDD), U9.14 (VDD)
- net y1: now also U4.1
- net y1': now also U4.2
- net y2: now also U4.3
- net y2': now also U4.4
- net y3: now also U4.5
- net y3': now also U4.6
- no-connect marks 1 -> 15
Other:
- sheet FullAdder: file FullAdder.kicad_sch -> fa1.kicad_sch
- sheet FullAdder ports: added none; removed GND, VCC
- sheet FullAdder1: file FullAdder.kicad_sch -> fa2.kicad_sch
- sheet FullAdder1 ports: added none; removed GND, VCC
- sheet FullAdder2: file FullAdder.kicad_sch -> fa3.kicad_sch
- sheet FullAdder2 ports: added none; removed GND, VCC
- sheet Multiplexer_3b: file multiplexer_3b.kicad_sch -> mux3b.kicad_sch
- sheet Multiplexer_3b ports: added none; removed GND, VCC
- sheet Multiplexer_6b1: file multiplexer_6b.kicad_sch -> mux6b1.kicad_sch
- sheet Multiplexer_6b1 ports: added none; removed GND, VCC
- sheet Multiplexer_6b2: file multiplexer_6b.kicad_sch -> mux6b2.kicad_sch
- sheet Multiplexer_6b2 ports: added none; removed GND, VCC

Commit message: Add files via upload
Parts:
- added D1, D10, D11, D12, D13, D14, D15, D2, D3, D4, D5, D6, D7, D8, D9: LED, Connector_PinHeader_2.54mm:PinHeader_1x02_P2.54mm_Vertical, symbol Device:LED
- added R1, R10, R11, R12, R13, R14, R2, R3, R4, R5, R6, R7, R8, R9: R, Connector_PinHeader_2.54mm:PinHeader_1x02_P2.54mm_Vertical, symbol Device:R
- added SW2, SW3, SW4, SW5, SW6, SW7, SW8, SW9: SW_DIP_x01, Connector_PinHeader_2.54mm:PinHeader_1x03_P2.54mm_Vertical, symbol Switch:SW_DIP_x01
- C1, C2: footprint Capacitor_THT:C_Rect_L7.0mm_W2.0mm_P5.00mm -> Capacitor_THT:C_Radial_D6.3mm_H5.0mm_P2.50mm
- SW1: footprint Connector_PinSocket_2.54mm:PinSocket_1x02_P2.54mm_Vertical -> Connector_PinHeader_2.54mm:PinHeader_1x03_P2.54mm_Vertical
Connections:
- net x3 is gone; now on net x2: J2.3 (Pin_3)
- net y3 is gone; now on net y2: J2.6 (Pin_6), U4.5
- net y3' is gone; now on net y2': U4.6
- net GND: now also D1.1 (K), R1.2, R10.2, R11.2, R12.2, R13.2, R14.2, R2.2, R3.2, R4.2, R5.2, R6.2, R7.2, R8.2, R9.2
- net VCC: now also D1.2 (A), SW2.1, SW3.1, SW4.1, SW5.1, SW6.1, SW7.1, SW8.1, SW9.1
- net ctrl_out0: now also D8.2 (A), SW8.2
- net ctrl_out1: now also D9.2 (A), SW9.2
- net x1: now also J2.2 (Pin_2), D3.2 (A), SW3.2; no longer J2.1 (Pin_1)
- net x2: now also D4.2 (A), SW4.2; no longer J2.2 (Pin_2)
- net y1: now also J2.5 (Pin_5), U4.3, D6.2 (A), SW6.2; no longer J2.4 (Pin_4), U4.1
- net y1': now also U4.4; no longer U4.2
- net y2: now also D7.2 (A), SW7.2; no longer J2.5 (Pin_5), U4.3
- net y2': no longer U4.4
- net Multiplexer_6b2/iout_0 renamed output 0
- net output 0: now also D10.2 (A)
- net Multiplexer_6b2/iout_1 renamed output 1
- net output 1: now also D11.2 (A)
- net Multiplexer_6b2/iout_2 renamed output 2
- net output 2: now also D12.2 (A)
- net Multiplexer_6b2/iout_3 renamed output 3
- net output 3: now also D13.2 (A)
- net Multiplexer_6b2/iout_4 renamed output 4
- net output 4: now also D14.2 (A)
- net Multiplexer_6b2/iout_5 renamed output 5
- net output 5: now also D15.2 (A)
- new net: D7.1 (K), R6.1
- new net: D3.1 (K), R2.1
- new net: D15.1 (K), R14.1
- new net: D4.1 (K), R3.1
- new net: D13.1 (K), R12.1
- new net: D6.1 (K), R5.1
- new net: D12.1 (K), R11.1
- new net: D5.1 (K), R4.1
- new net: D2.1 (K), R1.1
- new net: D14.1 (K), R13.1
- new net: D9.1 (K), R8.1
- new net: D11.1 (K), R10.1
- new net: D8.1 (K), R7.1
- new net: D10.1 (K), R9.1
- new net x0: D2.2 (A), J2.1 (Pin_1), SW2.2
- new net y0: D5.2 (A), J2.4 (Pin_4), SW5.2, U4.1
- new net y0': U4.2
Other:
- note added: "INPUT SELECTOR"
- note added: "OUTPUT LED DISPLAY"
- note added: "SELECT OUTPUT"
- moved on the sheet: J4, U4A, U4B
