File: DTS.kicad_sch (KiCad schematic)
At the start: 9 parts, among them J1 Conn_01x02_Pin, J2 Conn_01x06_Pin, J3 Conn_01x02_Pin, J4 Conn_01x06_Pin, SW1 SW_DIP_x01, U1 4069, U2 LM7805_TO220

Commit message: Add files via upload
Parts:
- removed U1: 4069, Package_DIP:CERDIP-14_W7.62mm_SideBrazed_LongPads_Socket, symbol 4xxx:4069
- added U1, U11, U12, U15, U16, U19, U2, U20, U23, U24, U25, U28, U29, U30, U34, U35, U38, U39, U41, U42, U44, U45, U47, U48, U6, U7: 4081, Package_DIP:CERDIP-14_W7.62mm_SideBrazed_LongPads_Socket, symbol 4xxx:4081
- added U10, U13, U17, U21, U26, U3, U31, U36, U40, U43, U46, U8: 4071, Package_DIP:CERDIP-14_W7.62mm_SideBrazed_LongPads_Socket, symbol 4xxx:4071
- added U14, U18, U22, U27, U32, U37, U4, U5, U9: 4069, Package_DIP:CERDIP-14_W7.62mm_SideBrazed_LongPads_Socket, symbol 4xxx:4069
- renumbered U2 to U49
Connections:
- net GND: now also U1.7 (VSS), U10.7 (VSS), U11.7 (VSS), U12.7 (VSS), U13.7 (VSS), U14.7 (VSS), U15.7 (VSS), U16.7 (VSS), U17.7 (VSS), U18.7 (VSS), U19.7 (VSS), U2.7 (VSS), U20.7 (VSS), U21.7 (VSS), U22.7 (VSS), U23.7 (VSS), U24.7 (VSS), U25.7 (VSS), U26.7 (VSS), U27.7 (VSS), U28.7 (VSS), U29.7 (VSS), U3.7 (VSS), U30.7 (VSS), U31.7 (VSS), U32.7 (VSS), U34.7 (VSS), U35.7 (VSS), U36.7 (VSS), U37.7 (VSS), U38.7 (VSS), U39.7 (VSS), U4.7 (VSS), U40.7 (VSS), U41.7 (VSS), U42.7 (VSS), U43.7 (VSS), U44.7 (VSS), U45.7 (VSS), U46.7 (VSS), U47.7 (VSS), U48.7 (VSS), U5.7 (VSS), U6.7 (VSS), U7.7 (VSS), U8.7 (VSS), U9.7 (VSS)
- net VCC: now also U1.14 (VDD), U10.14 (VDD), U11.14 (VDD), U12.14 (VDD), U13.14 (VDD), U14.14 (VDD), U15.14 (VDD), U16.14 (VDD), U17.14 (VDD), U18.14 (VDD), U19.14 (VDD), U2.14 (VDD), U20.14 (VDD), U21.14 (VDD), U22.14 (VDD), U23.14 (VDD), U24.14 (VDD), U25.14 (VDD), U26.14 (VDD), U27.14 (VDD), U28.14 (VDD), U29.14 (VDD), U3.14 (VDD), U30.14 (VDD), U31.14 (VDD), U32.14 (VDD), U34.14 (VDD), U35.14 (VDD), U36.14 (VDD), U37.14 (VDD), U38.14 (VDD), U39.14 (VDD), U4.14 (VDD), U40.14 (VDD), U41.14 (VDD), U42.14 (VDD), U43.14 (VDD), U44.14 (VDD), U45.14 (VDD), U46.14 (VDD), U47.14 (VDD), U48.14 (VDD), U5.14 (VDD), U6.14 (VDD), U7.14 (VDD), U8.14 (VDD), U9.14 (VDD)
- net y1: now also U4.1
- net y1': now also U4.2
- net y2: now also U4.3
- net y2': now also U4.4
- net y3: now also U4.5
- net y3': now also U4.6
- no-connect marks 1 -> 15
Other:
- sheet FullAdder ports: added none; removed GND, VCC
- sheet FullAdder1 ports: added none; removed GND, VCC
- sheet FullAdder2 ports: added none; removed GND, VCC
- sheet Multiplexer_3b ports: added none; removed GND, VCC
- sheet Multiplexer_6b1 ports: added none; removed GND, VCC
- sheet Multiplexer_6b2 ports: added none; removed GND, VCC

Commit message: Add files via upload
Parts:
- added D1, D10, D11, D12, D13, D14, D15, D2, D3, D4, D5, D6, D7, D8, D9: LED, Connector_PinHeader_2.54mm:PinHeader_1x02_P2.54mm_Vertical, symbol Device:LED
- added R1, R10, R11, R12, R13, R14, R2, R3, R4, R5, R6, R7, R8, R9: R, Connector_PinHeader_2.54mm:PinHeader_1x02_P2.54mm_Vertical, symbol Device:R
- added SW2, SW3, SW4, SW5, SW6, SW7, SW8, SW9: SW_DIP_x01, Connector_PinHeader_2.54mm:PinHeader_1x03_P2.54mm_Vertical, symbol Switch:SW_DIP_x01
- C1, C2: footprint Capacitor_THT:C_Rect_L7.0mm_W2.0mm_P5.00mm -> Capacitor_THT:C_Radial_D6.3mm_H5.0mm_P2.50mm
- SW1: footprint Connector_PinSocket_2.54mm:PinSocket_1x02_P2.54mm_Vertical -> Connector_PinHeader_2.54mm:PinHeader_1x03_P2.54mm_Vertical
Connections:
- net x3 is gone; now on net x2: J2.3 (Pin_3)
- net GND: now also D1.1 (K), R1.2, R10.2, R11.2, R12.2, R13.2, R14.2, R2.2, R3.2, R4.2, R5.2, R6.2, R7.2, R8.2, R9.2
- net VCC: now also D1.2 (A), SW2.1, SW3.1, SW4.1, SW5.1, SW6.1, SW7.1, SW8.1, SW9.1
- net ctrl_out0: now also D8.2 (A), SW8.2
- net ctrl_out1: now also D9.2 (A), SW9.2
- net x1: now also J2.2 (Pin_2), D3.2 (A), SW3.2; no longer J2.1 (Pin_1)
- net x2: now also D4.2 (A), SW4.2; no longer J2.2 (Pin_2)
- net y1: now also J2.5 (Pin_5), D6.2 (A), SW6.2; no longer J2.4 (Pin_4)
- net y2: now also J2.6 (Pin_6), D7.2 (A), SW7.2; no longer J2.5 (Pin_5)
- net Multiplexer_6b2/iout_0 renamed output 0
- net output 0: now also D10.2 (A)
- net Multiplexer_6b2/iout_1 renamed output 1
- net output 1: now also D11.2 (A)
- net Multiplexer_6b2/iout_2 renamed output 2
- net output 2: now also D12.2 (A)
- net Multiplexer_6b2/iout_3 renamed output 3
- net output 3: now also D13.2 (A)
- net Multiplexer_6b2/iout_4 renamed output 4
- net output 4: now also D14.2 (A)
- net Multiplexer_6b2/iout_5 renamed output 5
- net output 5: now also D15.2 (A)
- net y3 renamed y0
- net y0: now also J2.4 (Pin_4), D5.2 (A), SW5.2; no longer J2.6 (Pin_6)
- net y3' renamed y0'
- new net: D7.1 (K), R6.1
- new net: D3.1 (K), R2.1
- new net: D15.1 (K), R14.1
- new net: D4.1 (K), R3.1
- new net: D13.1 (K), R12.1
- new net: D6.1 (K), R5.1
- new net: D12.1 (K), R11.1
- new net: D5.1 (K), R4.1
- new net: D2.1 (K), R1.1
- new net: D14.1 (K), R13.1
- new net: D9.1 (K), R8.1
- new net: D11.1 (K), R10.1
- new net: D8.1 (K), R7.1
- new net: D10.1 (K), R9.1
- new net x0: D2.2 (A), J2.1 (Pin_1), SW2.2
Other:
- note added: "INPUT SELECTOR"
- note added: "OUTPUT LED DISPLAY"
- note added: "SELECT OUTPUT"
- moved on the sheet: J4, U4A, U4B, U4C

Commit message: Add files via upload
Connections:
- net y0: now also U4.1; no longer U4.5
- net y0': now also U4.2; no longer U4.6
- net y1: now also U4.3; no longer U4.1
- net y1': now also U4.4; no longer U4.2
- net y2: now also U4.5; no longer U4.3
- net y2': now also U4.6; no longer U4.4
Other:
- moved on the sheet: U4A, U4B, U4C
Changed lines of the file:
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@@
 	(wire
 		(pts
+			(xy 44.45 83.82) (xy 43.18 83.82)
+		)
+		(stroke
+			(width 0)
+			(type default)
+		)
+	)
+	(wire
+		(pts
 			(xy 162.56 85.09) (xy 161.29 85.09)
 		)
@@
 	(wire
 		(pts
+			(xy 44.45 67.31) (xy 43.18 67.31)
+		)
+		(stroke
+			(width 0)
+			(type default)
+		)
+	)
+	(wire
+		(pts
 			(xy 86.36 77.47) (xy 92.71 77.47)
 		)
@@
 	(wire
 		(pts
-			(xy 29.21 68.58) (xy 30.48 68.58)
+			(xy 26.67 100.33) (xy 29.21 100.33)
 		)
 		(stroke
@@
 	(wire
 		(pts
-			(xy 27.94 101.6) (xy 29.21 101.6)
+			(xy 26.67 83.82) (xy 27.94 83.82)
 		)
 		(stroke
@@
 	(wire
 		(pts
+			(xy 26.67 67.31) (xy 27.94 67.31)
+		)
+		(stroke
+			(width 0)
+			(type default)
+		)
+	)
+	(wire
+		(pts
 			(xy 204.47 125.73) (xy 205.74 125.73)
 		)
@@
 	(wire
 		(pts
+			(xy 45.72 100.33) (xy 44.45 100.33)
+		)
+		(stroke
+			(width 0)
+			(type default)
+		)
+	)
+	(wire
+		(pts
 			(xy 240.03 55.88) (xy 240.03 82.55)
 		)
@@
 		)
 	)
-	(label "y0'"
-		(at 45.72 68.58 0)
+	(label "y2'"
+		(at 45.72 100.33 0)
 		(effects
 			(font
@@
 		)
 	)
-	(label "y1'"
-		(at 44.45 85.09 0)
+	(label "y0'"
+		(at 44.45 67.31 0)
 		(effects
 			(font
@@
 		)
 	)
-	(label "y2'"
-		(at 44.45 101.6 0)
+	(label "y1'"
+		(at 44.45 83.82 0)
 		(effects
 			(font
@@
 		)
 	)
-	(global_label "y0"
+	(global_label "y2"
 		(shape input)
-		(at 29.21 68.58 180)
+		(at 26.67 100.33 180)
 		(fields_autoplaced yes)
 		(effects
@@
 		)
 		(property "Intersheetrefs" "${INTERSHEET_REFS}"
-			(at 24.0477 68.58 0)
+			(at 21.5077 100.33 0)
 			(hide yes)
 			(show_name no)
@@
 		)
 	)
-	(global_label "y2"
+	(global_label "y1"
 		(shape input)
-		(at 27.94 101.6 180)
+		(at 26.67 83.82 180)
 		(fields_autoplaced yes)
 		(effects
@@
 		)
 		(property "Intersheetrefs" "${INTERSHEET_REFS}"
-			(at 22.7777 101.6 0)
+			(at 21.5077 83.82 0)
 			(hide yes)
 			(show_name no)
@@
 		)
 	)
-	(global_label "y1"
+	(global_label "y0"
 		(shape input)
-		(at 29.21 85.09 180)
+		(at 26.67 67.31 180)
 		(fields_autoplaced yes)
 		(effects
@@
 		)
 		(property "Intersheetrefs" "${INTERSHEET_REFS}"
-			(at 24.0477 85.09 0)
+			(at 21.5077 67.31 0)
 			(hide yes)
 			(show_name no)
@@
 	(symbol
 		(lib_id "4xxx:4069")
-		(at 36.83 85.09 0)
+		(at 35.56 67.31 0)
 		(unit 1)
 		(body_style 1)
@@
 		(fields_autoplaced yes)
 		(property "Reference" "U4"
-			(at 36.83 76.2 0)
+			(at 35.56 58.42 0)
 			(show_name no)
 			(do_not_autoplace no)
@@
 		)
 		(property "Value" "4069"
-			(at 36.83 78.74 0)
+			(at 35.56 60.96 0)
 			(show_name no)
 			(do_not_autoplace no)
@@
 		)
 		(property "Footprint" "Package_DIP:CERDIP-14_W7.62mm_SideBrazed_LongPads_Socket"
-			(at 36.83 85.09 0)
+			(at 35.56 67.31 0)
 			(hide yes)
 			(show_name no)
@@
 		)
 		(property "Datasheet" "http://www.intersil.com/content/dam/Intersil/documents/cd40/cd4069ubms.pdf"
-			(at 36.83 85.09 0)
+			(at 35.56 67.31 0)
 			(hide yes)
 			(show_name no)
@@
 		)
 		(property "Description" "Hex inverter"
-			(at 36.83 85.09 0)
+			(at 35.56 67.31 0)
 			(hide yes)
 			(show_name no)
@@
 	(symbol
 		(lib_id "4xxx:4069")
-		(at 38.1 68.58 0)
+		(at 36.83 100.33 0)
 		(unit 3)
 		(body_style 1)
@@
 		(fields_autoplaced yes)
 		(property "Reference" "U4"
-			(at 38.1 59.69 0)
+			(at 36.83 91.44 0)
 			(show_name no)
 			(do_not_autoplace no)
@@
 		)
 		(property "Value" "4069"
-			(at 38.1 62.23 0)
+			(at 36.83 93.98 0)
 			(show_name no)
 			(do_not_autoplace no)
@@
 		)
 		(property "Footprint" "Package_DIP:CERDIP-14_W7.62mm_SideBrazed_LongPads_Socket"
-			(at 38.1 68.58 0)
+			(at 36.83 100.33 0)
 			(hide yes)
 			(show_name no)
@@
 		)
 		(property "Datasheet" "http://www.intersil.com/content/dam/Intersil/documents/cd40/cd4069ubms.pdf"
-			(at 38.1 68.58 0)
+			(at 36.83 100.33 0)
 			(hide yes)
 			(show_name no)
@@
 		)
 		(property "Description" "Hex inverter"
-			(at 38.1 68.58 0)
+			(at 36.83 100.33 0)
 			(hide yes)
 			(show_name no)
@@
 	(symbol
 		(lib_id "4xxx:4069")
-		(at 36.83 101.6 0)
+		(at 35.56 83.82 0)
 		(unit 2)
 		(body_style 1)
@@
 		(fields_autoplaced yes)
 		(property "Reference" "U4"
-			(at 36.83 92.71 0)
+			(at 35.56 74.93 0)
 			(show_name no)
 			(do_not_autoplace no)
@@
 		)
 		(property "Value" "4069"
-			(at 36.83 95.25 0)
+			(at 35.56 77.47 0)
 			(show_name no)
 			(do_not_autoplace no)
@@
 		)
 		(property "Footprint" "Package_DIP:CERDIP-14_W7.62mm_SideBrazed_LongPads_Socket"
-			(at 36.83 101.6 0)
+			(at 35.56 83.82 0)
 			(hide yes)
 			(show_name no)
@@
 		)
 		(property "Datasheet" "http://www.intersil.com/content/dam/Intersil/documents/cd40/cd4069ubms.pdf"
-			(at 36.83 101.6 0)
+			(at 35.56 83.82 0)
 			(hide yes)
 			(show_name no)
@@
 		)
 		(property "Description" "Hex inverter"
-			(at 36.83 101.6 0)
+			(at 35.56 83.82 0)
 			(hide yes)
 			(show_name no)

Commit message: Add files via upload
Changed lines of the file:
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@@
 	(wire
 		(pts
+			(xy -274.32 97.79) (xy -274.32 95.25)
+		)
+		(stroke
+			(width 0)
+			(type default)
+		)
+	)
+	(wire
+		(pts
 			(xy 129.54 223.52) (xy 137.16 223.52)
 		)
@@
 		)
 	)
-	(global_label "GND"
-		(shape input)
-		(at -274.32 95.25 0)
-		(fields_autoplaced yes)
-		(effects
-			(font
-				(size 1.27 1.27)
-			)
-			(justify left)
-		)
-		(property "Intersheetrefs" "${INTERSHEET_REFS}"
-			(at -267.4643 95.25 0)
-			(hide yes)
-			(show_name no)
-			(do_not_autoplace no)
-			(effects
-				(font
-					(size 1.27 1.27)
-				)
-				(justify left)
-			)
-		)
-	)
 	(global_label "VCC"
 		(shape input)
@@
 	)
 	(symbol
+		(lib_id "power:PWR_FLAG")
+		(at 62.23 165.1 0)
+		(unit 1)
+		(body_style 1)
+		(exclude_from_sim no)
+		(in_bom yes)
+		(on_board yes)
+		(in_pos_files yes)
+		(dnp no)
+		(fields_autoplaced yes)
+		(property "Reference" "#FLG01"
+			(at 62.23 163.195 0)
+			(hide yes)
+			(show_name no)
+			(do_not_autoplace no)
+			(effects
+				(font
+					(size 1.27 1.27)
+				)
+			)
+		)
+		(property "Value" "PWR_FLAG"
+			(at 62.23 160.02 0)
+			(show_name no)
+			(do_not_autoplace no)
+			(effects
+				(font
+					(size 1.27 1.27)
+				)
+			)
+		)
+		(property "Footprint" ""
+			(at 62.23 165.1 0)
+			(hide yes)
+			(show_name no)
+			(do_not_autoplace no)
+			(effects
+				(font
+					(size 1.27 1.27)
+				)
+			)
+		)
+		(property "Datasheet" ""
+			(at 62.23 165.1 0)
+			(hide yes)
+			(show_name no)
+			(do_not_autoplace no)
+			(effects
+				(font
+					(size 1.27 1.27)
+				)
+			)
+		)
+		(property "Description" "Special symbol for telling ERC where power comes from"
+			(at 62.23 165.1 0)
+			(hide yes)
+			(show_name no)
+			(do_not_autoplace no)
+			(effects
+				(font
+					(size 1.27 1.27)
+				)
+			)
+		)
+		(pin "1"
+		)
+		(instances
+			(project "DTS"
+				(path "/1bd2ca98-343e-4f04-8d6c-1f7257d9e9fe"
+					(reference "#FLG01")
+					(unit 1)
+				)
+			)
+		)
+	)
+	(symbol
 		(lib_id "4xxx:4081")
 		(at -210.82 82.55 0)
@@
 	)
 	(symbol
+		(lib_id "power:PWR_FLAG")
+		(at 62.23 180.34 180)
+		(unit 1)
+		(body_style 1)
+		(exclude_from_sim no)
+		(in_bom yes)
+		(on_board yes)
+		(in_pos_files yes)
+		(dnp no)
+		(fields_autoplaced yes)
+		(property "Reference" "#FLG02"
+			(at 62.23 182.245 0)
+			(hide yes)
+			(show_name no)
+			(do_not_autoplace no)
+			(effects
+				(font
+					(size 1.27 1.27)
+				)
+			)
+		)
+		(property "Value" "PWR_FLAG"
+			(at 62.23 185.42 0)
+			(show_name no)
+			(do_not_autoplace no)
+			(effects
+				(font
+					(size 1.27 1.27)
+				)
+			)
+		)
+		(property "Footprint" ""
+			(at 62.23 180.34 0)
+			(hide yes)
+			(show_name no)
+			(do_not_autoplace no)
+			(effects
+				(font
+					(size 1.27 1.27)
+				)
+			)
+		)
+		(property "Datasheet" ""
+			(at 62.23 180.34 0)
+			(hide yes)
+			(show_name no)
+			(do_not_autoplace no)
+			(effects
+				(font
+					(size 1.27 1.27)
+				)
+			)
+		)
+		(property "Description" "Special symbol for telling ERC where power comes from"
+			(at 62.23 180.34 0)
+			(hide yes)
+			(show_name no)
+			(do_not_autoplace no)
+			(effects
+				(font
+					(size 1.27 1.27)
+				)
+			)
+		)
+		(pin "1"
+		)
+		(instances
+			(project "DTS"
+				(path "/1bd2ca98-343e-4f04-8d6c-1f7257d9e9fe"
+					(reference "#FLG02")
+					(unit 1)
+				)
+			)
+		)
+	)
+	(symbol
 		(lib_id "4xxx:4069")
 		(at -168.91 187.96 0)
@@
 					(unit 1)
 				)
+			)
+		)
+	)
+	(symbol
+		(lib_id "power:GND")
+		(at -274.32 97.79 0)
+		(unit 1)
+		(body_style 1)
+		(exclude_from_sim no)
+		(in_bom yes)
+		(on_board yes)
+		(in_pos_files yes)
+		(dnp no)
+		(fields_autoplaced yes)
+		(property "Reference" "#PWR025"
+			(at -274.32 104.14 0)
+			(hide yes)
+			(show_name no)
+			(do_not_autoplace no)
+			(effects
+				(font
+					(size 1.27 1.27)
+				)
+			)
+		)
+		(property "Value" "GND"
+			(at -274.32 102.87 0)
+			(show_name no)
+			(do_not_autoplace no)
+			(effects
+				(font
+					(size 1.27 1.27)
+				)
+			)
+		)
+		(property "Footprint" ""
+			(at -274.32 97.79 0)
+			(hide yes)
+			(show_name no)
+			(do_not_autoplace no)
+			(effects
+				(font
+					(size 1.27 1.27)
+				)
+			)
+		)
+		(property "Datasheet" ""
+			(at -274.32 97.79 0)
+			(hide yes)
+			(show_name no)
+			(do_not_autoplace no)
+			(effects
+				(font
+					(size 1.27 1.27)
+				)
+			)
+		)
+		(property "Description" "Power symbol creates a global label with name \"GND\" , ground"
+			(at -274.32 97.79 0)
+			(hide yes)
+			(show_name no)
+			(do_not_autoplace no)
+			(effects
+				(font
+					(size 1.27 1.27)
+				)
+			)
+		)
+		(pin "1"
+		)
+		(instances
+			(project "DTS"
+				(path "/1bd2ca98-343e-4f04-8d6c-1f7257d9e9fe"
+					(reference "#PWR025")
+					(unit 1)
+				)

Commit message: Add files via upload
Other:
- moved on the sheet: U10C, U10D, U10E, U11E, U12E, U13E, U14G, U15E, U16E, U17E, U18G, U19E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
