File: fa1.kicad_sch (KiCad schematic)
At the start: 7 parts, among them U1 4081, U10 4071, U18 4069, U27 4069, U46 4071, U48 4081, U6 4081

Commit message: Add files via upload
Parts:
- removed U1, U48, U6: 4081, Package_DIP:CERDIP-14_W7.62mm_SideBrazed_LongPads_Socket, symbol 4xxx:4081
- removed U10, U46: 4071, Package_DIP:CERDIP-14_W7.62mm_SideBrazed_LongPads_Socket, symbol 4xxx:4071
- removed U18, U27: 4069, Package_DIP:CERDIP-14_W7.62mm_SideBrazed_LongPads_Socket, symbol 4xxx:4069
- added U11, U15: 4081, Package_DIP:CERDIP-14_W7.62mm_SideBrazed_LongPads_Socket, symbol 4xxx:4081
- added U3, U8: 4071, Package_DIP:CERDIP-14_W7.62mm_SideBrazed_LongPads_Socket, symbol 4xxx:4071
- added U4, U9: 4069, Package_DIP:CERDIP-14_W7.62mm_SideBrazed_LongPads_Socket, symbol 4xxx:4069
Connections:
- new net (xy' + x'y)': U15.1, U9.4
- new net c_in: U15.2, U15.6, U9.1
- new net c_in': U11.13, U9.2
- new net c_out: U3.11
- new net sum: U8.4
- new net temp1: U11.11, U8.5
- new net temp2: U15.3, U8.6
- new net temp3: U15.4, U3.13
- new net x: U11.1, U11.5, U4.11
- new net x': U11.9, U4.10
- new net x'y: U8.2
- new net xor_out: U11.12, U15.5, U8.3, U9.3
- new net xy: U11.3, U3.12
- new net xy': U11.10, U11.4, U8.1
- new net y: U11.2, U11.8, U4.13
- new net y': U11.6, U4.12

Commit message: Add files via upload
Connections:
- net x'y: now also U11.10
- net xy': no longer U11.10
Changed lines of the file:
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@@
 		)
 	)
-	(label "xy'"
+	(label "x'y"
 		(at 157.48 57.15 0)
 		(effects
