File: fa1.kicad_sch (KiCad schematic)
At the start: 4 parts, among them U3 4081, U4 4069, U5 4071, U6 4081

Commit message: Add files via upload
Parts:
- removed U3, U6: 4081, Package_DIP:CERDIP-14_W7.62mm_SideBrazed_LongPads_Socket, symbol 4xxx:4081
- removed unit 1 of U4
- removed unit 4 of U4
- removed unit 3 of U4
- removed unit 2 of U4
- removed unit 7 of U4
- removed U5: 4071, Package_DIP:CERDIP-14_W7.62mm_SideBrazed_LongPads_Socket, symbol 4xxx:4071
- added U11, U15: 4081, Package_DIP:CERDIP-14_W7.62mm_SideBrazed_LongPads_Socket, symbol 4xxx:4081
- added U3, U8: 4071, Package_DIP:CERDIP-14_W7.62mm_SideBrazed_LongPads_Socket, symbol 4xxx:4071
- added U9: 4069, Package_DIP:CERDIP-14_W7.62mm_SideBrazed_LongPads_Socket, symbol 4xxx:4069
Connections:
- net (xy' + x'y)': now also U15.1, U9.4; no longer U4.12
- net c_in: now also U15.2, U15.6, U9.1
- net c_in': now also U11.13, U9.2
- net c_out: now also U3.11
- net sum: now also U8.4
- net temp1: now also U11.11, U8.5
- net temp2: now also U15.3, U8.6
- net temp3: now also U15.4, U3.13
- net x: now also U4.11, U11.1, U11.5
- net x': now also U4.10, U11.9
- net x'y: now also U8.2
- net xor_out: now also U11.12, U15.5, U8.3, U9.3; no longer U4.13
- net xy: now also U11.3, U3.12
- net xy': now also U11.10, U11.4, U8.1
- net y: now also U4.13, U11.2, U11.8
- net y': now also U4.12, U11.6

Commit message: Add files via upload
Connections:
- net x'y: now also U11.10
- net xy': no longer U11.10
