File: fa3.kicad_sch (KiCad schematic)
At the start: 7 parts, among them U1 4081, U10 4071, U18 4069, U27 4069, U46 4071, U48 4081, U6 4081

Commit message: Add files via upload
Parts:
- removed U1, U48, U6: 4081, Package_DIP:CERDIP-14_W7.62mm_SideBrazed_LongPads_Socket, symbol 4xxx:4081
- removed U10, U46: 4071, Package_DIP:CERDIP-14_W7.62mm_SideBrazed_LongPads_Socket, symbol 4xxx:4071
- removed U18, U27: 4069, Package_DIP:CERDIP-14_W7.62mm_SideBrazed_LongPads_Socket, symbol 4xxx:4069
- added U13: 4071, Package_DIP:CERDIP-14_W7.62mm_SideBrazed_LongPads_Socket, symbol 4xxx:4071
- added U18: 4069, Package_DIP:CERDIP-14_W7.62mm_SideBrazed_LongPads_Socket, symbol 4xxx:4069
- added U24, U29: 4081, Package_DIP:CERDIP-14_W7.62mm_SideBrazed_LongPads_Socket, symbol 4xxx:4081
Connections:
- new net (xy' + x'y)': U18.8, U29.1
- new net c_in: U18.5, U29.2, U29.6
- new net c_in': U18.6, U24.13
- new net c_out: U13.11
- new net sum: U13.10
- new net temp1: U13.8, U24.11
- new net temp2: U13.9, U29.3
- new net temp3: U13.13, U29.4
- new net x: U18.1, U24.1, U24.5
- new net x': U18.2, U24.9
- new net x'y: U13.6
- new net xor_out: U13.4, U18.9, U24.12, U29.5
- new net xy: U13.12, U24.3
- new net xy': U13.5, U24.10, U24.4
- new net y: U18.3, U24.2, U24.8
- new net y': U18.4, U24.6

Commit message: Add files via upload
Connections:
- net x'y: now also U24.10
- net xy': no longer U24.10
Changed lines of the file:
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@@
+		)
+	)
+	(label "x'y"
+		(at 157.48 57.15 0)
+		(effects
+			(font
+				(size 1.27 1.27)
+			)
+			(justify left bottom)
 		)
 	)
@@
 		(effects
 			(font
-				(size 1.27 1.27)
-			)
-			(justify left bottom)
-		)
-	)
-	(label "xy'"
-		(at 157.48 57.15 0)
-		(effects
-			(font
