File: fa3.kicad_sch (KiCad schematic)
At the start: 4 parts, among them U11 4081, U12 4069, U13 4071, U14 4081

Commit message: Add files via upload
Parts:
- removed U11, U14: 4081, Package_DIP:CERDIP-14_W7.62mm_SideBrazed_LongPads_Socket, symbol 4xxx:4081
- removed U12: 4069, Package_DIP:CERDIP-14_W7.62mm_SideBrazed_LongPads_Socket, symbol 4xxx:4069
- removed unit 1 of U13
- removed unit 5 of U13
- added U18: 4069, Package_DIP:CERDIP-14_W7.62mm_SideBrazed_LongPads_Socket, symbol 4xxx:4069
- added U24, U29: 4081, Package_DIP:CERDIP-14_W7.62mm_SideBrazed_LongPads_Socket, symbol 4xxx:4081
Connections:
- net (xy' + x'y)': now also U18.8, U29.1
- net c_in: now also U18.5, U29.2, U29.6
- net c_in': now also U18.6, U24.13
- net c_out: now also U13.11; no longer U13.4
- net sum: now also U13.10; no longer U13.11
- net temp1: now also U13.8, U24.11; no longer U13.12
- net temp2: now also U13.9, U29.3; no longer U13.13
- net temp3: now also U13.13, U29.4; no longer U13.6
- net x: now also U18.1, U24.1, U24.5
- net x': now also U18.2, U24.9
- net x'y: now also U13.6; no longer U13.9
- net xor_out: now also U13.4, U18.9, U24.12, U29.5; no longer U13.10
- net xy: now also U13.12, U24.3; no longer U13.5
- net xy': now also U13.5, U24.10, U24.4; no longer U13.8
- net y: now also U18.3, U24.2, U24.8
- net y': now also U18.4, U24.6

Commit message: Add files via upload
Connections:
- net x'y: now also U24.10
- net xy': no longer U24.10
