File: fa6.kicad_sch (KiCad schematic)
At the start: 7 parts, among them U1 4081, U10 4071, U18 4069, U27 4069, U46 4071, U48 4081, U6 4081

Commit message: Add files via upload
Parts:
- removed U1, U48, U6: 4081, Package_DIP:CERDIP-14_W7.62mm_SideBrazed_LongPads_Socket, symbol 4xxx:4081
- removed U10, U46: 4071, Package_DIP:CERDIP-14_W7.62mm_SideBrazed_LongPads_Socket, symbol 4xxx:4071
- removed U18, U27: 4069, Package_DIP:CERDIP-14_W7.62mm_SideBrazed_LongPads_Socket, symbol 4xxx:4069
- added U22: 4069, Package_DIP:CERDIP-14_W7.62mm_SideBrazed_LongPads_Socket, symbol 4xxx:4069
- added U25, U30: 4081, Package_DIP:CERDIP-14_W7.62mm_SideBrazed_LongPads_Socket, symbol 4xxx:4081
- added U36, U40: 4071, Package_DIP:CERDIP-14_W7.62mm_SideBrazed_LongPads_Socket, symbol 4xxx:4071
Connections:
- new net (xy' + x'y)': U22.10, U30.8
- new net c_in: U22.9, U30.13, U30.9
- new net c_in': U22.8, U30.6
- new net c_out: U36.11
- new net sum: U36.10
- new net temp1: U30.4, U36.8
- new net temp2: U30.10, U36.9
- new net temp3: U30.11, U36.13
- new net x: U22.3, U25.5, U25.8
- new net x': U22.4, U25.13
- new net x'y: U40.2
- new net xor_out: U22.11, U30.12, U30.5, U40.3
- new net xy: U25.4, U36.12
- new net xy': U25.10, U25.11, U40.1
- new net y: U22.5, U25.12, U25.6
- new net y': U22.6, U25.9

Commit message: Add files via upload
Connections:
- net x'y: now also U25.11
- net xy': no longer U25.11
Changed lines of the file:
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@@
-		)
-	)
-	(label "xy'"
-		(at 157.48 57.15 0)
-		(effects
-			(font
-				(size 1.27 1.27)
-			)
-			(justify left bottom)
 		)
 	)
@@
 		(effects
 			(font
+				(size 1.27 1.27)
+			)
+			(justify left bottom)
+		)
+	)
+	(label "x'y"
+		(at 157.48 57.15 0)
+		(effects
+			(font
