File: fa6.kicad_sch (KiCad schematic)
At the start: 4 parts, among them U43 4081, U44 4069, U45 4071, U46 4081

Commit message: Add files via upload
Parts:
- removed U43, U46: 4081, Package_DIP:CERDIP-14_W7.62mm_SideBrazed_LongPads_Socket, symbol 4xxx:4081
- removed U44: 4069, Package_DIP:CERDIP-14_W7.62mm_SideBrazed_LongPads_Socket, symbol 4xxx:4069
- removed U45: 4071, Package_DIP:CERDIP-14_W7.62mm_SideBrazed_LongPads_Socket, symbol 4xxx:4071
- added U22: 4069, Package_DIP:CERDIP-14_W7.62mm_SideBrazed_LongPads_Socket, symbol 4xxx:4069
- added U25, U30: 4081, Package_DIP:CERDIP-14_W7.62mm_SideBrazed_LongPads_Socket, symbol 4xxx:4081
- added U36, U40: 4071, Package_DIP:CERDIP-14_W7.62mm_SideBrazed_LongPads_Socket, symbol 4xxx:4071
Connections:
- net (xy' + x'y)': now also U22.10, U30.8
- net c_in: now also U22.9, U30.13, U30.9
- net c_in': now also U22.8, U30.6
- net c_out: now also U36.11
- net sum: now also U36.10
- net temp1: now also U30.4, U36.8
- net temp2: now also U30.10, U36.9
- net temp3: now also U30.11, U36.13
- net x: now also U22.3, U25.5, U25.8
- net x': now also U22.4, U25.13
- net x'y: now also U40.2
- net xor_out: now also U22.11, U30.12, U30.5, U40.3
- net xy: now also U25.4, U36.12
- net xy': now also U25.10, U25.11, U40.1
- net y: now also U22.5, U25.12, U25.6
- net y': now also U22.6, U25.9

Commit message: Add files via upload
Connections:
- net x'y: now also U25.11
- net xy': no longer U25.11
