File: fa9.kicad_sch (KiCad schematic)
At the start: 7 parts, among them U1 4081, U10 4071, U18 4069, U27 4069, U46 4071, U48 4081, U6 4081

Commit message: Add files via upload
Parts:
- removed U1, U48, U6: 4081, Package_DIP:CERDIP-14_W7.62mm_SideBrazed_LongPads_Socket, symbol 4xxx:4081
- removed U10, U46: 4071, Package_DIP:CERDIP-14_W7.62mm_SideBrazed_LongPads_Socket, symbol 4xxx:4071
- removed U18, U27: 4069, Package_DIP:CERDIP-14_W7.62mm_SideBrazed_LongPads_Socket, symbol 4xxx:4069
- added U42, U45, U48: 4081, Package_DIP:CERDIP-14_W7.62mm_SideBrazed_LongPads_Socket, symbol 4xxx:4081
- added U43, U46: 4071, Package_DIP:CERDIP-14_W7.62mm_SideBrazed_LongPads_Socket, symbol 4xxx:4071
- added U5: 4069, Package_DIP:CERDIP-14_W7.62mm_SideBrazed_LongPads_Socket, symbol 4xxx:4069
Connections:
- new net (xy' + x'y)': U45.12, U5.10
- new net c_in: U45.13, U48.2, U5.9
- new net c_in': U45.9, U5.8
- new net c_out: U46.4
- new net sum: U46.3
- new net temp1: U45.10, U46.1
- new net temp2: U45.11, U46.2
- new net temp3: U46.6, U48.3
- new net x: U42.1, U45.1, U5.3
- new net x': U45.6, U5.4
- new net x'y: U43.13
- new net xor_out: U43.11, U45.8, U48.1, U5.11
- new net xy: U42.3, U46.5
- new net xy': U43.12, U45.3, U45.4
- new net y: U42.2, U45.5, U5.5
- new net y': U45.2, U5.6

Commit message: Add files via upload
Connections:
- net x'y: now also U45.4
- net xy': no longer U45.4
Changed lines of the file:
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@@
+		)
+	)
+	(label "x'y"
+		(at 157.48 57.15 0)
+		(effects
+			(font
+				(size 1.27 1.27)
+			)
+			(justify left bottom)
 		)
 	)
@@
 		(effects
 			(font
-				(size 1.27 1.27)
-			)
-			(justify left bottom)
-		)
-	)
-	(label "xy'"
-		(at 157.48 57.15 0)
-		(effects
-			(font
