File: fa9.kicad_sch (KiCad schematic)
At the start: 4 parts, among them U55 4081, U56 4069, U57 4071, U58 4081

Commit message: Add files via upload
Parts:
- removed U55, U58: 4081, Package_DIP:CERDIP-14_W7.62mm_SideBrazed_LongPads_Socket, symbol 4xxx:4081
- removed U56: 4069, Package_DIP:CERDIP-14_W7.62mm_SideBrazed_LongPads_Socket, symbol 4xxx:4069
- removed U57: 4071, Package_DIP:CERDIP-14_W7.62mm_SideBrazed_LongPads_Socket, symbol 4xxx:4071
- added U42, U45, U48: 4081, Package_DIP:CERDIP-14_W7.62mm_SideBrazed_LongPads_Socket, symbol 4xxx:4081
- added U43, U46: 4071, Package_DIP:CERDIP-14_W7.62mm_SideBrazed_LongPads_Socket, symbol 4xxx:4071
- added U5: 4069, Package_DIP:CERDIP-14_W7.62mm_SideBrazed_LongPads_Socket, symbol 4xxx:4069
Connections:
- net (xy' + x'y)': now also U45.12, U5.10
- net c_in: now also U45.13, U48.2, U5.9
- net c_in': now also U45.9, U5.8
- net c_out: now also U46.4
- net sum: now also U46.3
- net temp1: now also U45.10, U46.1
- net temp2: now also U45.11, U46.2
- net temp3: now also U46.6, U48.3
- net x: now also U42.1, U45.1, U5.3
- net x': now also U45.6, U5.4
- net x'y: now also U43.13
- net xor_out: now also U43.11, U45.8, U48.1, U5.11
- net xy: now also U42.3, U46.5
- net xy': now also U43.12, U45.3, U45.4
- net y: now also U42.2, U45.5, U5.5
- net y': now also U45.2, U5.6

Commit message: Add files via upload
Connections:
- net x'y: now also U45.4
- net xy': no longer U45.4
